File: ice-adq.kicad_pcb (KiCad board)
At the start: 2 copper layers, 85.7 x 60.3 mm, 5 parts

Commit message: Ubicación de componentes y algo de ruteado
Parts:
- removed XA101: Conn_Poncho2P_2x_20x2, footprint:Conn_Poncho_SinBorde
- added C1: 0.01uF, Capacitor_SMD:C_0805_2012Metric_Pad1.15x1.40mm_HandSolder, F.Cu at (-76.9, 82.5)
- added C10: 1nF, Capacitor_SMD:C_0805_2012Metric_Pad1.15x1.40mm_HandSolder, F.Cu at (-64.0, 83.7)
- added C11: 0.01uF, Capacitor_SMD:C_0805_2012Metric_Pad1.15x1.40mm_HandSolder, F.Cu at (-30.5, 86.7)
- added C12: 0.01uF, Capacitor_SMD:C_0805_2012Metric_Pad1.15x1.40mm_HandSolder, F.Cu at (-34.7, 95.0)
- added C13: 0.01uF, Capacitor_SMD:C_0805_2012Metric_Pad1.15x1.40mm_HandSolder, F.Cu at (-56.2, 121.2)
- added C14: 0.22uF, Capacitor_SMD:CP_Elec_6.3x3, F.Cu at (-80.0, 135.0)
- added C15: 0.01uF, Capacitor_SMD:C_0805_2012Metric_Pad1.15x1.40mm_HandSolder, F.Cu at (-73.0, 128.8)
- added C16: 0.01uF, Capacitor_SMD:C_0805_2012Metric_Pad1.15x1.40mm_HandSolder, F.Cu at (-61.7, 89.7)
- added C2: 0.01uF, Capacitor_SMD:C_0805_2012Metric_Pad1.15x1.40mm_HandSolder, F.Cu at (-98.6, 82.5)
- added C3: 0.01uF, Capacitor_SMD:C_0805_2012Metric_Pad1.15x1.40mm_HandSolder, F.Cu at (-87.9, 82.5)
- added C4: 0.01uF, Capacitor_SMD:C_0805_2012Metric_Pad1.15x1.40mm_HandSolder, F.Cu at (-51.0, 83.8)
- added C5: 0.01uF, Capacitor_SMD:C_0805_2012Metric_Pad1.15x1.40mm_HandSolder, F.Cu at (-46.5, 83.8)
- added C6: 0.01uF, Capacitor_SMD:C_0805_2012Metric_Pad1.15x1.40mm_HandSolder, F.Cu at (-45.0, 105.5)
- added C7: 0.01uF, Capacitor_SMD:C_0805_2012Metric_Pad1.15x1.40mm_HandSolder, F.Cu at (-47.5, 105.5)
- added C8: 0.01uF, Capacitor_SMD:C_0805_2012Metric_Pad1.15x1.40mm_HandSolder, F.Cu at (-53.0, 105.0)
- added C9: 0.01uF, Capacitor_SMD:C_0805_2012Metric_Pad1.15x1.40mm_HandSolder, F.Cu at (-64.8, 106.5)
- added J1: T_Admisión, TerminalBlock:TerminalBlock_bornier-2_P5.08mm, F.Cu at (-76.5, 73.8)
- added J2: T_Escape, TerminalBlock:TerminalBlock_bornier-2_P5.08mm, F.Cu at (-87.5, 73.8)
- added J3: T_Aceite, TerminalBlock:TerminalBlock_bornier-2_P5.08mm, F.Cu at (-98.5, 73.8)
- added J4: Sonda Lambda, TerminalBlock:TerminalBlock_bornier-2_P5.08mm, F.Cu at (-49.2, 73.8)
- added J5: Sens. Inductivo, TerminalBlock:TerminalBlock_bornier-3_P5.08mm, F.Cu at (-65.5, 73.8)
- added J6: Sens. Presión, TerminalBlock:TerminalBlock_bornier-2_P5.08mm, F.Cu at (-38.0, 73.8)
- added J7: BATT, TerminalBlock:TerminalBlock_bornier-2_P5.08mm, F.Cu at (-77.5, 144.5)
- added R1: 100ohm, Resistor_SMD:R_0805_2012Metric_Pad1.15x1.40mm_HandSolder, F.Cu at (-50.5, 80.3)
- added R10: R_US, Resistor_SMD:R_0805_2012Metric_Pad1.15x1.40mm_HandSolder, F.Cu at (-38.2, 93.5)
- added R11: R_US, Resistor_SMD:R_0805_2012Metric_Pad1.15x1.40mm_HandSolder, F.Cu at (-34.7, 92.5)
- added R2: 100ohm, Resistor_SMD:R_0805_2012Metric_Pad1.15x1.40mm_HandSolder, F.Cu at (-48.0, 80.3)
- added R3: 10k, Resistor_SMD:R_0805_2012Metric_Pad1.15x1.40mm_HandSolder, F.Cu at (-42.5, 105.5)
- added R4: 1.1k, Resistor_SMD:R_0805_2012Metric_Pad1.15x1.40mm_HandSolder, F.Cu at (-53.0, 110.0)
- added R5: 680, Resistor_SMD:R_0805_2012Metric_Pad1.15x1.40mm_HandSolder, F.Cu at (-53.0, 107.5)
- added R6: 10k, Resistor_SMD:R_0805_2012Metric_Pad1.15x1.40mm_HandSolder, F.Cu at (-64.5, 93.2)
- added R7: 10k, Resistor_SMD:R_0805_2012Metric_Pad1.15x1.40mm_HandSolder, F.Cu at (-62.8, 80.2)
- added R8: 10k, Resistor_SMD:R_0805_2012Metric_Pad1.15x1.40mm_HandSolder, F.Cu at (-65.2, 80.2)
- added R9: R_US, Resistor_SMD:R_0805_2012Metric_Pad1.15x1.40mm_HandSolder, F.Cu at (-34.0, 81.2)
- added U1: MAX31855, Package_SO:SOIC-8_3.9x4.9mm_P1.27mm, F.Cu at (-72.9, 84.0)
- added U2: MAX31855, Package_SO:SOIC-8_3.9x4.9mm_P1.27mm, F.Cu at (-83.9, 84.0)
- added U3: MAX31855, Package_SO:SOIC-8_3.9x4.9mm_P1.27mm, F.Cu at (-94.6, 84.0)
- added U4: LM9044, Package_LCC:PLCC-20_SMD-Socket, F.Cu at (-50.0, 93.6)
- added U5: LM358, Package_SO:SOIC-8_3.9x4.9mm_P1.27mm, F.Cu at (-59.2, 105.8)
- added U6: MAX9924, umax:UMAX10, F.Cu at (-64.7, 88.5)
- added U7: LM358, Package_SO:SOIC-8_3.9x4.9mm_P1.27mm, F.Cu at (-34.7, 86.7)
- added U8: hm10, Connector_PinHeader_2.54mm:PinHeader_1x05_P2.54mm_Vertical, F.Cu at (-56.2, 116.1)
- added U9: L7805, Package_TO_SOT_SMD:TO-263-3_TabPin4, F.Cu at (-80.0, 122.0)
- added XA1: Conn_Poncho2P_2x_20x2, footprint:Conn_Poncho_SinBorde, F.Cu at (-29.3, 99.1)
- moved G*** 13.6 mm to (116.4, 96.8)
- moved G*** 13.6 mm to (116.4, 121.6)
- moved G101 13.6 mm to (116.4, 109.5)
- moved MP? 13.6 mm to (149.4, 92.4)
Routing:
- net +12V: track 0.00 -> 16.8 mm
- net Net-(C4-Pad2): track 0.00 -> 11.3 mm
- net Net-(J6-Pad2): track 0.00 -> 11.3 mm
- net Net-(J5-Pad3): track 0.00 -> 10.3 mm
- net Net-(J3-Pad1): track 0.00 -> 9.99 mm
- net Net-(J2-Pad1): track 0.00 -> 9.88 mm
- net Net-(J1-Pad1): track 0.00 -> 9.88 mm
- net Net-(C4-Pad1): track 0.00 -> 9.11 mm
- net Net-(J2-Pad2): track 0.00 -> 7.90 mm
- net Net-(J1-Pad2): track 0.00 -> 7.90 mm
- net Net-(J3-Pad2): track 0.00 -> 7.80 mm
- net Net-(J4-Pad2): track 0.00 -> 7.77 mm
- net Net-(J4-Pad1): track 0.00 -> 6.07 mm
- net Net-(J5-Pad1): track 0.00 -> 5.93 mm
- net +5V: track 0.00 -> 4.48 mm
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- added copper zone on In2.Cu, net +5V
- added copper zone on In1.Cu, net GND
Other:
- board size 85.7 x 60.3 mm -> 86 x 84 mm
- copper layers 2 -> 4
