File: rpm.sch (KiCad schematic (older format))
At the start: 0 parts

Commit message: Primer rev esquematicos RPM y comunicaciones
Parts:
- added C?: 1nF, symbol Device:C_Small
- added J?: Screw_Terminal_01x03, symbol Connector:Screw_Terminal_01x03
- added R? (x3): 10k, symbol Device:R_US
- added U?: MAX9924, symbol MAX9924-27:MAX9924
Connections:
- net labels added: +5V, GND, RPM_PULSE
- wire segments 0 -> 30
Changed lines of the file:
@@
 EELAYER 26 0
 EELAYER END
-$Descr A4 11693 8268
+$Descr A4 8268 11693 portrait
 encoding utf-8
-Sheet 1 5
-Title ""
-Date ""
+Sheet 4 6
+Title "Interfaz sensor RPM"
+Date "2021-12-11"
 Rev ""
 Comp ""
 Comment1 ""
-Comment2 ""
-Comment3 ""
+Comment2 "Especialización en Sistemas Embebidos 2021 - FIUBA"
+Comment3 "Autor: Ignacio Moya"
 Comment4 ""
 $EndDescr
+$Comp
+L MAX9924-27:MAX9924 U?
+U 1 1 61B5B6E4
+P 4050 5550
+F 0 "U?" H 4050 6215 50  0000 C CNN
+F 1 "MAX9924" H 4050 6124 50  0000 C CNN
+F 2 "" H 4050 5550 50  0001 C CNN
+F 3 "" H 4050 5550 50  0001 C CNN
+	1    4050 5550
+	-1   0    0    -1
+$EndComp
+$Comp
+L Device:R_US R?
+U 1 1 61B5B7AB
+P 5150 5050
+F 0 "R?" V 5050 5050 50  0000 C CNN
+F 1 "10k" V 5250 5050 50  0000 C CNN
+F 2 "" V 5190 5040 50  0001 C CNN
+F 3 "~" H 5150 5050 50  0001 C CNN
+	1    5150 5050
+	0    1    1    0
+$EndComp
+$Comp
+L Device:R_US R?
+U 1 1 61B5B80C
+P 5150 5450
+F 0 "R?" V 5050 5450 50  0000 C CNN
+F 1 "10k" V 5250 5450 50  0000 C CNN
+F 2 "" V 5190 5440 50  0001 C CNN
+F 3 "~" H 5150 5450 50  0001 C CNN
+	1    5150 5450
+	0    1    1    0
+$EndComp
+$Comp
+L Device:R_US R?
+U 1 1 61B5B826
+P 3100 5400
+F 0 "R?" H 3168 5446 50  0000 L CNN
+F 1 "10k" H 3168 5355 50  0000 L CNN
+F 2 "" V 3140 5390 50  0001 C CNN
+F 3 "~" H 3100 5400 50  0001 C CNN
+	1    3100 5400
+	1    0    0    -1
+$EndComp
+$Comp
+L Device:C_Small C?
+U 1 1 61B5B942
+P 4750 5250
+F 0 "C?" H 4842 5296 50  0000 L CNN
+F 1 "1nF" H 4842 5205 50  0000 L CNN
+F 2 "" H 4750 5250 50  0001 C CNN
+F 3 "~" H 4750 5250 50  0001 C CNN
+	1    4750 5250
+	1    0    0    -1
+$EndComp
+$Comp
+L basico-rescue:GND #PWR?
+U 1 1 61B5BC42
+P 3450 6250
+F 0 "#PWR?" H 3450 6000 50  0001 C CNN
+F 1 "GND" H 3455 6077 50  0000 C CNN
+F 2 "" H 3450 6250 50  0000 C CNN
+F 3 "" H 3450 6250 50  0000 C CNN
+	1    3450 6250
+	1    0    0    -1
+$EndComp
+Wire Wire Line
+	3550 5950 3450 5950
+$Comp
+L basico-rescue:+5V #PWR?
+U 1 1 61B5BF66
+P 3100 5050
+F 0 "#PWR?" H 3100 4900 50  0001 C CNN
+F 1 "+5V" H 3115 5223 50  0000 C CNN
+F 2 "" H 3100 5050 50  0000 C CNN
+F 3 "" H 3100 5050 50  0000 C CNN
+	1    3100 5050
+	1    0    0    -1
+$EndComp
+Text HLabel 2850 5750 0    50   Input ~ 0
+RPM_PULSE
+Wire Wire Line
+	3450 5950 3450 6150
+Wire Wire Line
+	4650 5950 4650 6150
+Wire Wire Line
+	4650 6150 3450 6150
+Wire Wire Line
+	4550 5950 4650 5950
+Connection ~ 3450 6150
+Wire Wire Line
+	3450 6150 3450 6250
+Wire Wire Line
+	4550 5750 4650 5750
+Wire Wire Line
+	4650 5750 4650 5950
+Connection ~ 4650 5950
+Wire Wire Line
+	3550 5350 3450 5350
+Wire Wire Line
+	3450 5350 3450 5950
+Connection ~ 3450 5950
+Wire Wire Line
+	2850 5750 3100 5750
+Wire Wire Line
+	3100 5550 3100 5750
+Connection ~ 3100 5750
+Wire Wire Line
+	3100 5750 3550 5750
+Wire Wire Line
+	3550 5150 3100 5150
+Wire Wire Line
+	3100 5150 3100 5250
+Wire Wire Line
+	3100 5050 3100 5150
+Connection ~ 3100 5150
+Wire Wire Line
+	4550 5150 4750 5150
+Wire Wire Line
+	4550 5350 4750 5350
+Wire Wire Line
+	4750 5350 4750 5450
+Wire Wire Line
+	4750 5450 5000 5450
+Connection ~ 4750 5350
+Wire Wire Line
+	4750 5150 4750 5050
+Wire Wire Line
+	4750 5050 5000 5050
+Connection ~ 4750 5150
+$Comp
+L Connector:Screw_Terminal_01x03 J?
+U 1 1 61B5E81F
+P 5850 5250
+F 0 "J?" H 5930 5246 50  0000 L CNN
+F 1 "Screw_Terminal_01x03" H 5930 5201 50  0001 L CNN
+F 2 "" H 5850 5250 50  0001 C CNN
+F 3 "~" H 5850 5250 50  0001 C CNN
+	1    5850 5250
+	1    0    0    -1
+$EndComp
+Wire Wire Line
+	5300 5050 5400 5050
+Wire Wire Line
+	5400 5050 5400 5150
+Wire Wire Line
+	5300 5450 5400 5450
+Wire Wire Line
+	5400 5450 5400 5350
+$Comp
+L basico-rescue:GND #PWR?
+U 1 1 61B5EE58
+P 5550 5550
+F 0 "#PWR?" H 5550 5300 50  0001 C CNN
+F 1 "GND" H 5555 5377 50  0000 C CNN
+F 2 "" H 5550 5550 50  0000 C CNN
+F 3 "" H 5550 5550 50  0000 C CNN
+	1    5550 5550
+	1    0    0    -1
+$EndComp
+Wire Wire Line
+	5400 5350 5650 5350
+Wire Wire Line
+	5400 5150 5650 5150
+Wire Wire Line
+	5650 5250 5550 5250
+Wire Wire Line
+	5550 5250 5550 5550
 $EndSCHEMATC

Commit message: Esquematicos mayormente terminados, falta sub-hoja edu ciaa, fuentes de alimentacion y poner valores a los componentes
Other:
- note added: "- El integrado MAX9924 permite ser operado en hasta cuatro modos de\noperación diferentes. En este esquemático, el módo de operación sele-\nccionado es el A2. Esto quiere decir que tiene activadas la detección\npor cero, detección de pico adaptativa y utiliza la referencia de voltaje\ninterna. Según la hoja de datos, este modo de operación es el más\nrobusto y sencillo ya que reduce la cantidad d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"
- note added: "Interfaz sensor inductivo con EDU-CIAA"
Changed lines of the file:
@@
 Date "2021-12-11"
 Rev ""
-Comp ""
-Comment1 ""
-Comment2 "Especialización en Sistemas Embebidos 2021 - FIUBA"
-Comment3 "Autor: Ignacio Moya"
+Comp "Autor: Ignacio Moya"
+Comment1 "Especialización en Sistemas Embebidos 2021 - FIUBA"
+Comment2 ""
+Comment3 ""
 Comment4 ""
 $EndDescr
@@
 Wire Wire Line
 	5550 5250 5550 5550
+Wire Notes Line
+	2300 4600 6100 4600
+Wire Notes Line
+	6100 4600 6100 6550
+Wire Notes Line
+	6100 6550 2300 6550
+Wire Notes Line
+	2300 6550 2300 4600
+Text Notes 2300 4550 0    50   ~ 0
+Interfaz sensor inductivo con EDU-CIAA
+Text Notes 2350 7150 0    50   ~ 0
+-  El integrado MAX9924 permite ser operado en hasta cuatro modos de\noperación diferentes. En este esquemático, el módo de operación sele-\nccionado es el A2. Esto quiere decir que tiene activadas la detección\npor cero, detección de pico adaptativa y utiliza la referencia de voltaje\ninterna. Según la hoja de datos, este modo de operación es el más\nrobusto y sencillo ya que reduce la cantidad de componentes externos.
 $EndSCHEMATC

Commit message: Se agrego esquematico de fuentes y se corrigieron errores de ERC
Parts:
- gave numbers to parts that had none: 6
Connections:
- no-connect marks 0 -> 2
Changed lines of the file:
@@
 $Descr A4 8268 11693 portrait
 encoding utf-8
-Sheet 4 6
+Sheet 4 8
 Title "Interfaz sensor RPM"
-Date "2021-12-11"
-Rev ""
+Date "2021-12-18"
+Rev "1.0"
 Comp "Autor: Ignacio Moya"
 Comment1 "Especialización en Sistemas Embebidos 2021 - FIUBA"
@@
 $EndDescr
 $Comp
-L MAX9924-27:MAX9924 U?
+L MAX9924-27:MAX9924 U6
 U 1 1 61B5B6E4
 P 4050 5550
-F 0 "U?" H 4050 6215 50  0000 C CNN
+F 0 "U6" H 4050 6215 50  0000 C CNN
 F 1 "MAX9924" H 4050 6124 50  0000 C CNN
 F 2 "" H 4050 5550 50  0001 C CNN
@@
 $EndComp
 $Comp
-L Device:R_US R?
+L Device:R_US R7
 U 1 1 61B5B7AB
 P 5150 5050
-F 0 "R?" V 5050 5050 50  0000 C CNN
+F 0 "R7" V 5050 5050 50  0000 C CNN
 F 1 "10k" V 5250 5050 50  0000 C CNN
 F 2 "" V 5190 5040 50  0001 C CNN
@@
 $EndComp
 $Comp
-L Device:R_US R?
+L Device:R_US R8
 U 1 1 61B5B80C
 P 5150 5450
-F 0 "R?" V 5050 5450 50  0000 C CNN
+F 0 "R8" V 5050 5450 50  0000 C CNN
 F 1 "10k" V 5250 5450 50  0000 C CNN
 F 2 "" V 5190 5440 50  0001 C CNN
@@
 $EndComp
 $Comp
-L Device:R_US R?
+L Device:R_US R6
 U 1 1 61B5B826
 P 3100 5400
-F 0 "R?" H 3168 5446 50  0000 L CNN
+F 0 "R6" H 3168 5446 50  0000 L CNN
 F 1 "10k" H 3168 5355 50  0000 L CNN
 F 2 "" V 3140 5390 50  0001 C CNN
@@
 $EndComp
 $Comp
-L Device:C_Small C?
+L Device:C_Small C10
 U 1 1 61B5B942
 P 4750 5250
-F 0 "C?" H 4842 5296 50  0000 L CNN
+F 0 "C10" H 4842 5296 50  0000 L CNN
 F 1 "1nF" H 4842 5205 50  0000 L CNN
 F 2 "" H 4750 5250 50  0001 C CNN
@@
 $EndComp
 $Comp
-L basico-rescue:GND #PWR?
+L basico-rescue:GND #PWR030
 U 1 1 61B5BC42
 P 3450 6250
-F 0 "#PWR?" H 3450 6000 50  0001 C CNN
+F 0 "#PWR030" H 3450 6000 50  0001 C CNN
 F 1 "GND" H 3455 6077 50  0000 C CNN
 F 2 "" H 3450 6250 50  0000 C CNN
@@
 	3550 5950 3450 5950
 $Comp
-L basico-rescue:+5V #PWR?
+L basico-rescue:+5V #PWR029
 U 1 1 61B5BF66
 P 3100 5050
-F 0 "#PWR?" H 3100 4900 50  0001 C CNN
+F 0 "#PWR029" H 3100 4900 50  0001 C CNN
 F 1 "+5V" H 3115 5223 50  0000 C CNN
 F 2 "" H 3100 5050 50  0000 C CNN
@@
 	1    0    0    -1
 $EndComp
-Text HLabel 2850 5750 0    50   Input ~ 0
+Text HLabel 2850 5750 0    50   Output ~ 0
 RPM_PULSE
 Wire Wire Line
@@
 Connection ~ 4750 5150
 $Comp
-L Connector:Screw_Terminal_01x03 J?
+L Connector:Screw_Terminal_01x03 J5
 U 1 1 61B5E81F
 P 5850 5250
-F 0 "J?" H 5930 5246 50  0000 L CNN
+F 0 "J5" H 5930 5246 50  0000 L CNN
 F 1 "Screw_Terminal_01x03" H 5930 5201 50  0001 L CNN
 F 2 "" H 5850 5250 50  0001 C CNN
@@
 	5400 5450 5400 5350
 $Comp
-L basico-rescue:GND #PWR?
+L basico-rescue:GND #PWR031
 U 1 1 61B5EE58
 P 5550 5550
-F 0 "#PWR?" H 5550 5300 50  0001 C CNN
+F 0 "#PWR031" H 5550 5300 50  0001 C CNN
 F 1 "GND" H 5555 5377 50  0000 C CNN
 F 2 "" H 5550 5550 50  0000 C CNN
@@
 Text Notes 2350 7150 0    50   ~ 0
 -  El integrado MAX9924 permite ser operado en hasta cuatro modos de\noperación diferentes. En este esquemático, el módo de operación sele-\nccionado es el A2. Esto quiere decir que tiene activadas la detección\npor cero, detección de pico adaptativa y utiliza la referencia de voltaje\ninterna. Según la hoja de datos, este modo de operación es el más\nrobusto y sencillo ya que reduce la cantidad de componentes externos.
+NoConn ~ 4550 5550
+NoConn ~ 3550 5550
 $EndSCHEMATC

Commit message: Correccion de errores y se designaron huellas a casi todos los componentes
Parts:
- added C16: 0.01uF, Capacitor_SMD:C_0805_2012Metric_Pad1.15x1.40mm_HandSolder, symbol Device:C_Small
- C10: footprint (none) -> Capacitor_SMD:C_0805_2012Metric_Pad1.15x1.40mm_HandSolder
- J5: value Screw_Terminal_01x03 -> Sens. Inductivo; footprint (none) -> TerminalBlock:TerminalBlock_bornier-3_P5.08mm
- R6, R7, R8: footprint (none) -> Resistor_SMD:R_0805_2012Metric_Pad1.15x1.40mm_HandSolder
- U6: footprint (none) -> umax:UMAX10
Connections:
- wire segments 30 -> 33
Other:
- note added: "- El integrado MAX9924 permite ser configurado en hasta cuatro modos de\noperación diferentes. En este esquemático, el módo de operación sele-\nccionado es el A2. Esto quiere decir que tiene activadas la detección\npor cero, detección de pico adaptativa y utiliza la referencia de voltaje\ninterna. Según la hoja de datos, este modo de operación es el más\nrobusto y sencillo ya que reduce la cantid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"
- note removed: "- El integrado MAX9924 permite ser operado en hasta cuatro modos de\noperación diferentes. En este esquemático, el módo de operación sele-\nccionado es el A2. Esto quiere decir que tiene activadas la detección\npor cero, detección de pico adaptativa y utiliza la referencia de voltaje\ninterna. Según la hoja de datos, este modo de operación es el más\nrobusto y sencillo ya que reduce la cantidad d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"
Changed lines of the file:
@@
 Sheet 4 8
 Title "Interfaz sensor RPM"
-Date "2021-12-18"
+Date "2021-12-19"
 Rev "1.0"
 Comp "Autor: Ignacio Moya"
@@
 F 0 "U6" H 4050 6215 50  0000 C CNN
 F 1 "MAX9924" H 4050 6124 50  0000 C CNN
-F 2 "" H 4050 5550 50  0001 C CNN
+F 2 "umax:UMAX10" H 4050 5550 50  0001 C CNN
 F 3 "" H 4050 5550 50  0001 C CNN
 	1    4050 5550
@@
 F 0 "R7" V 5050 5050 50  0000 C CNN
 F 1 "10k" V 5250 5050 50  0000 C CNN
-F 2 "" V 5190 5040 50  0001 C CNN
+F 2 "Resistor_SMD:R_0805_2012Metric_Pad1.15x1.40mm_HandSolder" V 5190 5040 50  0001 C CNN
 F 3 "~" H 5150 5050 50  0001 C CNN
 	1    5150 5050
@@
 F 0 "R8" V 5050 5450 50  0000 C CNN
 F 1 "10k" V 5250 5450 50  0000 C CNN
-F 2 "" V 5190 5440 50  0001 C CNN
+F 2 "Resistor_SMD:R_0805_2012Metric_Pad1.15x1.40mm_HandSolder" V 5190 5440 50  0001 C CNN
 F 3 "~" H 5150 5450 50  0001 C CNN
 	1    5150 5450
@@
 F 0 "R6" H 3168 5446 50  0000 L CNN
 F 1 "10k" H 3168 5355 50  0000 L CNN
-F 2 "" V 3140 5390 50  0001 C CNN
+F 2 "Resistor_SMD:R_0805_2012Metric_Pad1.15x1.40mm_HandSolder" V 3140 5390 50  0001 C CNN
 F 3 "~" H 3100 5400 50  0001 C CNN
 	1    3100 5400
@@
 F 0 "C10" H 4842 5296 50  0000 L CNN
 F 1 "1nF" H 4842 5205 50  0000 L CNN
-F 2 "" H 4750 5250 50  0001 C CNN
+F 2 "Capacitor_SMD:C_0805_2012Metric_Pad1.15x1.40mm_HandSolder" H 4750 5250 50  0001 C CNN
 F 3 "~" H 4750 5250 50  0001 C CNN
 	1    4750 5250
@@
 P 5850 5250
 F 0 "J5" H 5930 5246 50  0000 L CNN
-F 1 "Screw_Terminal_01x03" H 5930 5201 50  0001 L CNN
-F 2 "" H 5850 5250 50  0001 C CNN
+F 1 "Sens. Inductivo" H 5500 5500 50  0000 L CNN
+F 2 "TerminalBlock:TerminalBlock_bornier-3_P5.08mm" H 5850 5250 50  0001 C CNN
 F 3 "~" H 5850 5250 50  0001 C CNN
 	1    5850 5250
@@
 Interfaz sensor inductivo con EDU-CIAA
 Text Notes 2350 7150 0    50   ~ 0
--  El integrado MAX9924 permite ser operado en hasta cuatro modos de\noperación diferentes. En este esquemático, el módo de operación sele-\nccionado es el A2. Esto quiere decir que tiene activadas la detección\npor cero, detección de pico adaptativa y utiliza la referencia de voltaje\ninterna. Según la hoja de datos, este modo de operación es el más\nrobusto y sencillo ya que reduce la cantidad de componentes externos.
+-  El integrado MAX9924 permite ser configurado en hasta cuatro modos de\noperación diferentes. En este esquemático, el módo de operación sele-\nccionado es el A2. Esto quiere decir que tiene activadas la detección\npor cero, detección de pico adaptativa y utiliza la referencia de voltaje\ninterna. Según la hoja de datos, este modo de operación es el más\nrobusto y sencillo ya que reduce la cantidad de componentes externos.
 NoConn ~ 4550 5550
 NoConn ~ 3550 5550
+$Comp
+L Device:C_Small C16
+U 1 1 61C1397B
+P 2650 5300
+F 0 "C16" H 2742 5346 50  0000 L CNN
+F 1 "0.01uF" H 2742 5255 50  0000 L CNN
+F 2 "Capacitor_SMD:C_0805_2012Metric_Pad1.15x1.40mm_HandSolder" H 2650 5300 50  0001 C CNN
+F 3 "~" H 2650 5300 50  0001 C CNN
+	1    2650 5300
+	1    0    0    -1
+$EndComp
+$Comp
+L basico-rescue:GND #PWR0109
+U 1 1 61C13D81
+P 2650 5450
+F 0 "#PWR0109" H 2650 5200 50  0001 C CNN
+F 1 "GND" H 2655 5277 50  0000 C CNN
+F 2 "" H 2650 5450 50  0000 C CNN
+F 3 "" H 2650 5450 50  0000 C CNN
+	1    2650 5450
+	1    0    0    -1
+$EndComp
+Wire Wire Line
+	2650 5450 2650 5400
+Wire Wire Line
+	2650 5200 2650 5150
+Wire Wire Line
+	2650 5150 3100 5150
 $EndSCHEMATC
