File: oxigeno.sch (KiCad schematic (older format))
At the start: 0 parts

Commit message: avances en el esquematico del amplificador de sonda lambda
Parts:
- added C? (x5): 0.01uF, symbol Device:C_Small
- added J?: Screw_Terminal_01x02, symbol Connector:Screw_Terminal_01x02
- added R?: 10k, symbol Device:R_Small
- added R? (x2): 100ohm, symbol Device:R_Small
- added U?: LM9044, symbol Oxigen_Sensor:LM9044
Connections:
- net labels added: +12V, +5V, GND
- wire segments 0 -> 29

Commit message: Esquematicos mayormente terminados, falta sub-hoja edu ciaa, fuentes de alimentacion y poner valores a los componentes
Parts:
- removed R?: 10k, symbol Device:R_Small
- removed R? (x2): 100ohm, symbol Device:R_Small
- added C?: 0.01uF, symbol Device:C_Small
- added R? (x2): 100ohm, symbol Device:R_US
- added R?: 10k, symbol Device:R_US
- added R? (x2): R_US, symbol Device:R_US
- added U? (x3): LM358, symbol Amplifier_Operational:LM358
- J?: value Screw_Terminal_01x02 -> Sonda Lambda
Connections:
- net labels added: O2_OUT
- wire segments 29 -> 56
Other:
- note added: "Amplificador de sensor de oxígeno"
- note added: "Circuito interfaz sensor de oxígeno y EDU-CIAA"
- note added: "Etapa amplificadora A=0.6 (5v a 3.3v)"

Commit message: Se agrego esquematico de fuentes y se corrigieron errores de ERC
Parts:
- removed U?: LM9044, symbol Oxigen_Sensor:LM9044
- added U4: LM9044, symbol Oxigen_Sensor:LM9044
- gave numbers to parts that had none: 13
Changed lines of the file:
@@
 $Descr A4 8268 11693 portrait
 encoding utf-8
-Sheet 3 6
+Sheet 3 8
 Title "Amplificador de sensor de oxígeno"
 Date "2021-12-18"
-Rev ""
+Rev "1.0"
 Comp "Autor: Ignacio Moya"
 Comment1 "Especialización en Sistemas Embebidos 2021 - FIUBA"
@@
 $EndDescr
 $Comp
-L power:+12V #PWR?
+L power:+12V #PWR021
 U 1 1 6027D6DE
 P 2850 4200
-F 0 "#PWR?" H 2850 4050 50  0001 C CNN
+F 0 "#PWR021" H 2850 4050 50  0001 C CNN
 F 1 "+12V" H 2865 4373 50  0000 C CNN
 F 2 "" H 2850 4200 50  0001 C CNN
@@
 $EndComp
 $Comp
-L power:+5V #PWR?
+L power:+5V #PWR023
 U 1 1 6027D709
 P 3050 4200
-F 0 "#PWR?" H 3050 4050 50  0001 C CNN
+F 0 "#PWR023" H 3050 4050 50  0001 C CNN
 F 1 "+5V" H 3065 4373 50  0000 C CNN
 F 2 "" H 3050 4200 50  0001 C CNN
@@
 $EndComp
 $Comp
-L power:GND #PWR?
+L power:GND #PWR022
 U 1 1 6027D73B
 P 2850 6050
-F 0 "#PWR?" H 2850 5800 50  0001 C CNN
+F 0 "#PWR022" H 2850 5800 50  0001 C CNN
 F 1 "GND" H 2855 5877 50  0000 C CNN
 F 2 "" H 2850 6050 50  0001 C CNN
@@
 $EndComp
 $Comp
-L Device:C_Small C?
+L Device:C_Small C4
 U 1 1 6027D844
 P 2000 5250
-F 0 "C?" H 2092 5296 50  0000 L CNN
+F 0 "C4" H 2092 5296 50  0000 L CNN
 F 1 "0.01uF" H 2092 5205 50  0000 L CNN
 F 2 "" H 2000 5250 50  0001 C CNN
@@
 $EndComp
 $Comp
-L power:GND #PWR?
+L power:GND #PWR019
 U 1 1 6027D8AF
 P 2000 5750
-F 0 "#PWR?" H 2000 5500 50  0001 C CNN
+F 0 "#PWR019" H 2000 5500 50  0001 C CNN
 F 1 "GND" H 2005 5577 50  0000 C CNN
 F 2 "" H 2000 5750 50  0001 C CNN
@@
 $EndComp
 $Comp
-L Device:C_Small C?
+L Device:C_Small C6
 U 1 1 6027D8D8
 P 2650 4650
-F 0 "C?" V 2550 4650 50  0000 C CNN
+F 0 "C6" V 2550 4650 50  0000 C CNN
 F 1 "0.01uF" V 2750 4650 50  0000 C CNN
 F 2 "" H 2650 4650 50  0001 C CNN
@@
 $EndComp
 $Comp
-L power:GND #PWR?
+L power:GND #PWR020
 U 1 1 6027D930
 P 2350 4700
-F 0 "#PWR?" H 2350 4450 50  0001 C CNN
+F 0 "#PWR020" H 2350 4450 50  0001 C CNN
 F 1 "GND" H 2355 4527 50  0000 C CNN
 F 2 "" H 2350 4700 50  0001 C CNN
@@
 $EndComp
 $Comp
-L Oxigen_Sensor:LM9044 U?
-U 1 1 6027E1C9
-P 2850 5250
-F 0 "U?" H 3250 5500 50  0000 L CNN
-F 1 "LM9044" H 3250 5400 50  0000 L CNN
-F 2 "" H 2850 5250 50  0001 C CNN
-F 3 "" H 2850 5250 50  0001 C CNN
-	1    2850 5250
-	1    0    0    -1
-$EndComp
-$Comp
-L Device:C_Small C?
+L Device:C_Small C5
 U 1 1 6027E2F3
 P 2000 5550
-F 0 "C?" H 2092 5596 50  0000 L CNN
+F 0 "C5" H 2092 5596 50  0000 L CNN
 F 1 "0.01uF" H 2092 5505 50  0000 L CNN
 F 2 "" H 2000 5550 50  0001 C CNN
@@
 	2000 5750 2000 5650
 $Comp
-L Device:C_Small C?
+L Device:C_Small C7
 U 1 1 6027E605
 P 3000 5850
-F 0 "C?" H 3092 5896 50  0000 L CNN
+F 0 "C7" H 3092 5896 50  0000 L CNN
 F 1 "0.01uF" H 3092 5805 50  0000 L CNN
 F 2 "" H 3000 5850 50  0001 C CNN
@@
 Wire Wire Line
 	2750 4650 2850 4650
-Wire Wire Line
-	2850 4650 2850 4800
-$Comp
-L Connector:Screw_Terminal_01x02 J?
+$Comp
+L Connector:Screw_Terminal_01x02 J4
 U 1 1 6027F2A5
 P 1000 5300
-F 0 "J?" H 920 4975 50  0000 C CNN
+F 0 "J4" H 920 4975 50  0000 C CNN
 F 1 "Sonda Lambda" H 920 5066 50  0000 C CNN
 F 2 "" H 1000 5300 50  0001 C CNN
@@
 	-1   0    0    1
 $EndComp
-Wire Wire Line
-	1550 5100 1550 5200
-Wire Wire Line
-	1400 5200 1200 5200
-Wire Wire Line
-	1200 5300 1400 5300
-Wire Wire Line
-	1550 5300 1550 5400
-$Comp
-L Device:C_Small C?
+$Comp
+L Device:C_Small C8
 U 1 1 6027FB98
 P 3400 5400
-F 0 "C?" H 3492 5446 50  0000 L CNN
+F 0 "C8" H 3492 5446 50  0000 L CNN
 F 1 "0.01uF" H 3492 5355 50  0000 L CNN
 F 2 "" H 3400 5400 50  0001 C CNN
@@
 $EndComp
 $Comp
-L power:GND #PWR?
+L power:GND #PWR024
 U 1 1 6027FC2C
 P 3400 5600
-F 0 "#PWR?" H 3400 5350 50  0001 C CNN
+F 0 "#PWR024" H 3400 5350 50  0001 C CNN
 F 1 "GND" H 3405 5427 50  0000 C CNN
 F 2 "" H 3400 5600 50  0001 C CNN
@@
 	3400 5500 3400 5600
 $Comp
-L Device:R_US R?
+L Device:R_US R1
 U 1 1 61BF348E
 P 1750 5100
-F 0 "R?" V 1650 5100 50  0000 C CNN
+F 0 "R1" V 1650 5100 50  0000 C CNN
 F 1 "100ohm" V 1850 5100 50  0000 C CNN
 F 2 "" V 1790 5090 50  0001 C CNN
@@
 $EndComp
 $Comp
-L Device:R_US R?
+L Device:R_US R2
 U 1 1 61BF3601
 P 1750 5400
-F 0 "R?" V 1650 5400 50  0000 C CNN
+F 0 "R2" V 1650 5400 50  0000 C CNN
 F 1 "100ohm" V 1850 5400 50  0000 C CNN
 F 2 "" V 1790 5390 50  0001 C CNN
@@
 $EndComp
 $Comp
-L Device:R_US R?
+L Device:R_US R3
 U 1 1 61BF3746
 P 2850 4400
-F 0 "R?" H 2750 4400 50  0000 C CNN
+F 0 "R3" H 2750 4400 50  0000 C CNN
 F 1 "10k" H 2950 4400 50  0000 C CNN
 F 2 "" V 2890 4390 50  0001 C CNN
@@
 Wire Wire Line
 	2850 4550 2850 4650
-Connection ~ 2850 4650
 Wire Wire Line
 	2850 4200 2850 4250
-Wire Wire Line
-	1550 5100 1600 5100
-Wire Wire Line
-	1550 5400 1600 5400
 Wire Wire Line
 	1900 5400 2000 5400
@@
 Connection ~ 2000 5100
 Wire Wire Line
-	1400 5300 1550 5300
-Connection ~ 1400 5300
-Wire Wire Line
-	1400 5200 1550 5200
-Connection ~ 1400 5200
-Wire Wire Line
 	2350 5400 2000 5400
 $Comp
-L Amplifier_Operational:LM358 U?
+L Amplifier_Operational:LM358 U5
 U 1 1 61BF972E
 P 4450 5350
-F 0 "U?" H 4450 4983 50  0000 C CNN
+F 0 "U5" H 4450 4983 50  0000 C CNN
 F 1 "LM358" H 4450 5074 50  0000 C CNN
 F 2 "" H 4450 5350 50  0001 C CNN
@@
 $EndComp
 $Comp
-L Amplifier_Operational:LM358 U?
+L Amplifier_Operational:LM358 U5
 U 2 1 61BF97AD
 P 5550 5450
-F 0 "U?" H 5550 5083 50  0000 C CNN
+F 0 "U5" H 5550 5083 50  0000 C CNN
 F 1 "LM358" H 5550 5174 50  0000 C CNN
 F 2 "" H 5550 5450 50  0001 C CNN
@@
 $EndComp
 $Comp
-L Amplifier_Operational:LM358 U?
+L Amplifier_Operational:LM358 U5
 U 3 1 61BF982A
 P 7300 5400
-F 0 "U?" H 7258 5446 50  0000 L CNN
+F 0 "U5" H 7258 5446 50  0000 L CNN
 F 1 "LM358" H 7258 5355 50  0000 L CNN
 F 2 "" H 7300 5400 50  0001 C CNN
@@
 	4050 5250 4150 5250
 $Comp
-L power:GND #PWR?
+L power:GND #PWR025
 U 1 1 61BFA9F5
 P 4050 5550
-F 0 "#PWR?" H 4050 5300 50  0001 C CNN
+F 0 "#PWR025" H 4050 5300 50  0001 C CNN
 F 1 "GND" H 4055 5377 50  0000 C CNN
 F 2 "" H 4050 5550 50  0001 C CNN
@@
 	4050 5450 4050 5550
 $Comp
-L Device:R_US R?
+L Device:R_US R5
 U 1 1 61BFB624
 P 5600 4950
-F 0 "R?" V 5395 4950 50  0000 C CNN
+F 0 "R5" V 5395 4950 50  0000 C CNN
 F 1 "R_US" V 5486 4950 50  0000 C CNN
 F 2 "" V 5640 4940 50  0001 C CNN
@@
 $EndComp
 $Comp
-L Device:R_US R?
+L Device:R_US R4
 U 1 1 61BFB6A9
 P 5000 5350
-F 0 "R?" V 4795 5350 50  0000 C CNN
+F 0 "R4" V 4795 5350 50  0000 C CNN
 F 1 "R_US" V 4886 5350 50  0000 C CNN
 F 2 "" V 5040 5340 50  0001 C CNN
@@
 	5950 5450 5850 5450
 $Comp
-L power:GND #PWR?
+L power:GND #PWR026
 U 1 1 61BFD69D
 P 5200 5650
-F 0 "#PWR?" H 5200 5400 50  0001 C CNN
+F 0 "#PWR026" H 5200 5400 50  0001 C CNN
 F 1 "GND" H 5205 5477 50  0000 C CNN
 F 2 "" H 5200 5650 50  0001 C CNN
@@
 Connection ~ 4050 5250
 $Comp
-L Device:C_Small C?
+L Device:C_Small C9
 U 1 1 61C026B4
 P 6950 5400
-F 0 "C?" H 7042 5446 50  0000 L CNN
+F 0 "C9" H 7042 5446 50  0000 L CNN
 F 1 "0.01uF" H 7042 5355 50  0000 L CNN
 F 2 "" H 6950 5400 50  0001 C CNN
@@
 	6950 5700 7200 5700
 $Comp
-L power:GND #PWR?
+L power:GND #PWR028
 U 1 1 61C04594
 P 7200 5750
-F 0 "#PWR?" H 7200 5500 50  0001 C CNN
+F 0 "#PWR028" H 7200 5500 50  0001 C CNN
 F 1 "GND" H 7205 5577 50  0000 C CNN
 F 2 "" H 7200 5750 50  0001 C CNN
@@
 $EndComp
 $Comp
-L power:+5V #PWR?
+L power:+5V #PWR027
 U 1 1 61C048CF
 P 7200 5050
-F 0 "#PWR?" H 7200 4900 50  0001 C CNN
+F 0 "#PWR027" H 7200 4900 50  0001 C CNN
 F 1 "+5V" H 7215 5223 50  0000 C CNN
 F 2 "" H 7200 5050 50  0001 C CNN
@@
 Text Notes 650  3500 0    50   ~ 0
 Circuito interfaz sensor de oxígeno y EDU-CIAA
+Wire Wire Line
+	1600 5400 1400 5400
+Wire Wire Line
+	1250 5400 1250 5300
+Wire Wire Line
+	1250 5300 1200 5300
+Wire Wire Line
+	1200 5200 1250 5200
+Wire Wire Line
+	1250 5200 1250 5100
+Wire Wire Line
+	1250 5100 1400 5100
+Connection ~ 1400 5400
+Wire Wire Line
+	1400 5400 1250 5400
+Connection ~ 1400 5100
+Wire Wire Line
+	1400 5100 1600 5100
+Wire Wire Line
+	2850 4650 2850 4800
+Connection ~ 2850 4650
+$Comp
+L Oxigen_Sensor:LM9044 U4
+U 1 1 61C66195
+P 2850 5250
+F 0 "U4" H 3250 5550 50  0000 L CNN
+F 1 "LM9044" H 3250 5450 50  0000 L CNN
+F 2 "" H 2850 5250 50  0001 C CNN
+F 3 "" H 2850 5250 50  0001 C CNN
+	1    2850 5250
+	1    0    0    -1
+$EndComp
 $EndSCHEMATC

Commit message: Correccion de errores y se designaron huellas a casi todos los componentes
Parts:
- C4, C5, C6, C7, C8, C9: footprint (none) -> Capacitor_SMD:C_0805_2012Metric_Pad1.15x1.40mm_HandSolder
- R1, R2, R3: footprint (none) -> Resistor_SMD:R_0805_2012Metric_Pad1.15x1.40mm_HandSolder
- R4: value R_US -> 1.1k; footprint (none) -> Resistor_SMD:R_0805_2012Metric_Pad1.15x1.40mm_HandSolder
- R5: value R_US -> 680; footprint (none) -> Resistor_SMD:R_0805_2012Metric_Pad1.15x1.40mm_HandSolder
- U4: footprint (none) -> Package_LCC:PLCC-20_SMD-Socket
- U5: footprint (none) -> Package_SO:SOIC-8_3.9x4.9mm_P1.27mm
Connections:
- wire segments 56 -> 51
- no-connect marks 0 -> 1
Other:
- note added: "Etapa seguidora de voltaje y atenuación A=0.6 (5v a 3.3v)"
- note removed: "Etapa amplificadora A=0.6 (5v a 3.3v)"
- moved on the sheet: U5A, U5B, U5C

Commit message: Ubicación de componentes y algo de ruteado
Connections:
- wire segments 51 -> 54
Changed lines of the file:
@@
 L Connector:Screw_Terminal_01x02 J4
 U 1 1 6027F2A5
-P 1000 5300
-F 0 "J4" H 920 4975 50  0000 C CNN
-F 1 "Sonda Lambda" H 920 5066 50  0000 C CNN
-F 2 "" H 1000 5300 50  0001 C CNN
-F 3 "~" H 1000 5300 50  0001 C CNN
-	1    1000 5300
-	-1   0    0    1
+P 1000 5200
+F 0 "J4" H 1000 5350 50  0000 C CNN
+F 1 "Sonda Lambda" H 1000 4900 50  0000 C CNN
+F 2 "" H 1000 5200 50  0001 C CNN
+F 3 "~" H 1000 5200 50  0001 C CNN
+	1    1000 5200
+	-1   0    0    -1
 $EndComp
 $Comp
@@
 	6450 4150 6400 4150
 Wire Wire Line
-	6400 4150 6400 4350
+	6400 4150 6400 4250
 Wire Wire Line
 	6400 4350 6450 4350
@@
 	3400 5250 4350 5250
 Connection ~ 3400 5250
+$Comp
+L power:GND #PWR0110
+U 1 1 61BFA1FD
+P 6300 4300
+F 0 "#PWR0110" H 6300 4050 50  0001 C CNN
+F 1 "GND" H 6305 4127 50  0000 C CNN
+F 2 "" H 6300 4300 50  0001 C CNN
+F 3 "" H 6300 4300 50  0001 C CNN
+	1    6300 4300
+	1    0    0    -1
+$EndComp
+Wire Wire Line
+	6300 4300 6300 4250
+Wire Wire Line
+	6300 4250 6400 4250
+Connection ~ 6400 4250
+Wire Wire Line
+	6400 4250 6400 4350
 $EndSCHEMATC

Commit message: Se cambio pack de 7805 y de 9044
Parts:
- J4: footprint (none) -> TerminalBlock:TerminalBlock_bornier-2_P5.08mm
- U4: footprint Package_LCC:PLCC-20_SMD-Socket -> Package_LCC:PLCC-20
Changed lines of the file:
@@
 F 0 "J4" H 1000 5350 50  0000 C CNN
 F 1 "Sonda Lambda" H 1000 4900 50  0000 C CNN
-F 2 "" H 1000 5200 50  0001 C CNN
+F 2 "TerminalBlock:TerminalBlock_bornier-2_P5.08mm" H 1000 5200 50  0001 C CNN
 F 3 "~" H 1000 5200 50  0001 C CNN
 	1    1000 5200
@@
 F 0 "U4" H 3250 5550 50  0000 L CNN
 F 1 "LM9044" H 3250 5450 50  0000 L CNN
-F 2 "Package_LCC:PLCC-20_SMD-Socket" H 2850 5250 50  0001 C CNN
+F 2 "Package_LCC:PLCC-20" H 2850 5250 50  0001 C CNN
 F 3 "" H 2850 5250 50  0001 C CNN
 	1    2850 5250
