File: termocuplas.sch (KiCad schematic (older format))
At the start: 6 parts

Commit message: avances en el esquematico del amplificador de sonda lambda
Parts:
- added J? (x3): Screw_Terminal_01x02, symbol Connector:Screw_Terminal_01x02
Connections:
- wire segments 37 -> 43
Changed lines of the file:
@@
 Wire Wire Line
 	4500 5400 4750 5400
+$Comp
+L Connector:Screw_Terminal_01x02 J?
+U 1 1 601FF299
+P 3000 3850
+F 0 "J?" H 2920 3525 50  0000 C CNN
+F 1 "Screw_Terminal_01x02" H 2920 3616 50  0000 C CNN
+F 2 "" H 3000 3850 50  0001 C CNN
+F 3 "~" H 3000 3850 50  0001 C CNN
+	1    3000 3850
+	-1   0    0    1
+$EndComp
+$Comp
+L Connector:Screw_Terminal_01x02 J?
+U 1 1 601FF30D
+P 3050 4650
+F 0 "J?" H 2970 4325 50  0000 C CNN
+F 1 "Screw_Terminal_01x02" H 2970 4416 50  0000 C CNN
+F 2 "" H 3050 4650 50  0001 C CNN
+F 3 "~" H 3050 4650 50  0001 C CNN
+	1    3050 4650
+	-1   0    0    1
+$EndComp
+$Comp
+L Connector:Screw_Terminal_01x02 J?
+U 1 1 601FF365
+P 3100 5450
+F 0 "J?" H 3020 5125 50  0000 C CNN
+F 1 "Screw_Terminal_01x02" H 3020 5216 50  0000 C CNN
+F 2 "" H 3100 5450 50  0001 C CNN
+F 3 "~" H 3100 5450 50  0001 C CNN
+	1    3100 5450
+	-1   0    0    1
+$EndComp
+Wire Wire Line
+	3200 3750 3800 3750
+Wire Wire Line
+	3200 3850 3800 3850
+Wire Wire Line
+	3250 4550 3800 4550
+Wire Wire Line
+	3250 4650 3800 4650
+Wire Wire Line
+	3300 5350 3800 5350
+Wire Wire Line
+	3300 5450 3800 5450
 $EndSCHEMATC

Commit message: Esquematicos mayormente terminados, falta sub-hoja edu ciaa, fuentes de alimentacion y poner valores a los componentes
Parts:
- J?: value Screw_Terminal_01x02 -> T_Admisión
- J?: value Screw_Terminal_01x02 -> T_Escape
- J?: value Screw_Terminal_01x02 -> T_Aceite
Other:
- note added: "Alimentación y capacitores de desacople"
- note added: "Circuitos de amplificación y conversión de señal"

Commit message: Se agrego esquematico de fuentes y se corrigieron errores de ERC
Parts:
- removed U? (x3): MAX31855, symbol Amplifier_Thermocouple:MAX31855
- added U1, U2, U3: MAX31855, symbol Amplifier_Thermocouple:MAX31855
- gave numbers to parts that had none: 6
Changed lines of the file:
@@
 $Descr A4 8268 11693 portrait
 encoding utf-8
-Sheet 2 6
+Sheet 2 8
 Title "Amplificadores de termocuplas"
-Date "2021-02-07"
-Rev "R0"
+Date "2021-12-18"
+Rev "1.0"
 Comp "Autor: Ignacio Moya"
 Comment1 "Especialización en Sistemas Embebidos 2021 - FIUBA"
@@
 $EndDescr
 $Comp
-L Amplifier_Thermocouple:MAX31855 U?
-U 1 1 601FE82E
-P 4450 3750
-F 0 "U?" H 4450 4125 50  0000 C CNN
-F 1 "MAX31855" H 4450 4034 50  0000 C CNN
-F 2 "" H 4450 3750 50  0001 C CNN
-F 3 "" H 4450 3750 50  0001 C CNN
-	1    4450 3750
-	1    0    0    -1
-$EndComp
-$Comp
-L Amplifier_Thermocouple:MAX31855 U?
-U 1 1 601FE86C
-P 4450 4550
-F 0 "U?" H 4450 4925 50  0000 C CNN
-F 1 "MAX31855" H 4450 4834 50  0000 C CNN
-F 2 "" H 4450 4550 50  0001 C CNN
-F 3 "" H 4450 4550 50  0001 C CNN
-	1    4450 4550
-	1    0    0    -1
-$EndComp
-$Comp
-L Amplifier_Thermocouple:MAX31855 U?
-U 1 1 601FE8BD
-P 4450 5350
-F 0 "U?" H 4450 5725 50  0000 C CNN
-F 1 "MAX31855" H 4450 5634 50  0000 C CNN
-F 2 "" H 4450 5350 50  0001 C CNN
-F 3 "" H 4450 5350 50  0001 C CNN
-	1    4450 5350
-	1    0    0    -1
-$EndComp
-$Comp
-L Device:C_Small C?
+L Device:C_Small C1
 U 1 1 601FEC0E
 P 3700 6750
-F 0 "C?" H 3608 6704 50  0000 R CNN
+F 0 "C1" H 3608 6704 50  0000 R CNN
 F 1 "C_Small" H 3608 6795 50  0000 R CNN
 F 2 "" H 3700 6750 50  0001 C CNN
@@
 $EndComp
 $Comp
-L Device:C_Small C?
+L Device:C_Small C2
 U 1 1 601FEC5F
 P 4200 6750
-F 0 "C?" H 4108 6704 50  0000 R CNN
+F 0 "C2" H 4108 6704 50  0000 R CNN
 F 1 "C_Small" H 4108 6795 50  0000 R CNN
 F 2 "" H 4200 6750 50  0001 C CNN
@@
 $EndComp
 $Comp
-L Device:C_Small C?
+L Device:C_Small C3
 U 1 1 601FEC9C
 P 4650 6750
-F 0 "C?" H 4558 6704 50  0000 R CNN
+F 0 "C3" H 4558 6704 50  0000 R CNN
 F 1 "C_Small" H 4558 6795 50  0000 R CNN
 F 2 "" H 4650 6750 50  0001 C CNN
@@
 ACT_CS
 $Comp
-L power:+3V3 #PWR?
+L power:+3V3 #PWR03
 U 1 1 601FEEB4
 P 3950 3500
-F 0 "#PWR?" H 3950 3350 50  0001 C CNN
+F 0 "#PWR03" H 3950 3350 50  0001 C CNN
 F 1 "+3V3" H 3965 3673 50  0000 C CNN
 F 2 "" H 3950 3500 50  0001 C CNN
@@
 $EndComp
 $Comp
-L power:GND #PWR?
+L power:GND #PWR04
 U 1 1 601FEF21
 P 4000 5650
-F 0 "#PWR?" H 4000 5400 50  0001 C CNN
+F 0 "#PWR04" H 4000 5400 50  0001 C CNN
 F 1 "GND" H 4005 5477 50  0000 C CNN
 F 2 "" H 4000 5650 50  0001 C CNN
@@
 	4100 5200 3950 5200
 $Comp
-L power:GND #PWR?
+L power:GND #PWR018
 U 1 1 601FF433
 P 4200 7050
-F 0 "#PWR?" H 4200 6800 50  0001 C CNN
+F 0 "#PWR018" H 4200 6800 50  0001 C CNN
 F 1 "GND" H 4205 6877 50  0000 C CNN
 F 2 "" H 4200 7050 50  0001 C CNN
@@
 	4200 7050 4200 6850
 $Comp
-L power:+3V3 #PWR?
+L power:+3V3 #PWR013
 U 1 1 601FFCA9
 P 4200 6500
-F 0 "#PWR?" H 4200 6350 50  0001 C CNN
+F 0 "#PWR013" H 4200 6350 50  0001 C CNN
 F 1 "+3V3" H 4215 6673 50  0000 C CNN
 F 2 "" H 4200 6500 50  0001 C CNN
@@
 	4800 5400 5050 5400
 $Comp
-L Connector:Screw_Terminal_01x02 J?
+L Connector:Screw_Terminal_01x02 J1
 U 1 1 601FF299
 P 3300 3850
-F 0 "J?" H 3220 3525 50  0000 C CNN
+F 0 "J1" H 3220 3525 50  0000 C CNN
 F 1 "T_Admisión" H 3220 3616 50  0000 C CNN
 F 2 "" H 3300 3850 50  0001 C CNN
@@
 $EndComp
 $Comp
-L Connector:Screw_Terminal_01x02 J?
+L Connector:Screw_Terminal_01x02 J2
 U 1 1 601FF30D
 P 3350 4650
-F 0 "J?" H 3270 4325 50  0000 C CNN
+F 0 "J2" H 3270 4325 50  0000 C CNN
 F 1 "T_Escape" H 3270 4416 50  0000 C CNN
 F 2 "" H 3350 4650 50  0001 C CNN
@@
 $EndComp
 $Comp
-L Connector:Screw_Terminal_01x02 J?
+L Connector:Screw_Terminal_01x02 J3
 U 1 1 601FF365
 P 3400 5450
-F 0 "J?" H 3320 5125 50  0000 C CNN
+F 0 "J3" H 3320 5125 50  0000 C CNN
 F 1 "T_Aceite" H 3320 5216 50  0000 C CNN
 F 2 "" H 3400 5450 50  0001 C CNN
@@
 	-1   0    0    1
 $EndComp
-Wire Wire Line
-	3500 3750 4100 3750
-Wire Wire Line
-	3500 3850 4100 3850
-Wire Wire Line
-	3550 4550 4100 4550
-Wire Wire Line
-	3550 4650 4100 4650
-Wire Wire Line
-	3600 5350 4100 5350
-Wire Wire Line
-	3600 5450 4100 5450
 Wire Notes Line
 	2850 3150 5550 3150
@@
 Wire Notes Line
 	2600 7500 2600 2900
+$Comp
+L Amplifier_Thermocouple:MAX31855 U1
+U 1 1 61C66817
+P 4450 3750
+F 0 "U1" H 4450 4125 50  0000 C CNN
+F 1 "MAX31855" H 4450 4034 50  0000 C CNN
+F 2 "" H 4450 3750 50  0001 C CNN
+F 3 "" H 4450 3750 50  0001 C CNN
+	1    4450 3750
+	1    0    0    -1
+$EndComp
+$Comp
+L Amplifier_Thermocouple:MAX31855 U3
+U 1 1 61C66899
+P 4450 5350
+F 0 "U3" H 4450 5725 50  0000 C CNN
+F 1 "MAX31855" H 4450 5634 50  0000 C CNN
+F 2 "" H 4450 5350 50  0001 C CNN
+F 3 "" H 4450 5350 50  0001 C CNN
+	1    4450 5350
+	1    0    0    -1
+$EndComp
+$Comp
+L Amplifier_Thermocouple:MAX31855 U2
+U 1 1 61C66976
+P 4450 4550
+F 0 "U2" H 4450 4925 50  0000 C CNN
+F 1 "MAX31855" H 4450 4834 50  0000 C CNN
+F 2 "" H 4450 4550 50  0001 C CNN
+F 3 "" H 4450 4550 50  0001 C CNN
+	1    4450 4550
+	1    0    0    -1
+$EndComp
+Wire Wire Line
+	3600 5450 4100 5450
+Wire Wire Line
+	3600 5350 4100 5350
+Wire Wire Line
+	3550 4650 4100 4650
+Wire Wire Line
+	3550 4550 4100 4550
+Wire Wire Line
+	3500 3850 4100 3850
+Wire Wire Line
+	3500 3750 4100 3750
 $EndSCHEMATC

Commit message: Correccion de errores y se designaron huellas a casi todos los componentes
Parts:
- C1, C2, C3: value C_Small -> 0.01uF; footprint (none) -> Capacitor_SMD:C_0805_2012Metric_Pad1.15x1.40mm_HandSolder
- J1, J2, J3: footprint (none) -> TerminalBlock:TerminalBlock_bornier-2_P5.08mm
- U1, U2, U3: footprint (none) -> Package_SO:SOIC-8_3.9x4.9mm_P1.27mm
Changed lines of the file:
@@
 Sheet 2 8
 Title "Amplificadores de termocuplas"
-Date "2021-12-18"
+Date "2021-12-19"
 Rev "1.0"
 Comp "Autor: Ignacio Moya"
@@
 P 3700 6750
 F 0 "C1" H 3608 6704 50  0000 R CNN
-F 1 "C_Small" H 3608 6795 50  0000 R CNN
-F 2 "" H 3700 6750 50  0001 C CNN
+F 1 "0.01uF" H 3608 6795 50  0000 R CNN
+F 2 "Capacitor_SMD:C_0805_2012Metric_Pad1.15x1.40mm_HandSolder" H 3700 6750 50  0001 C CNN
 F 3 "~" H 3700 6750 50  0001 C CNN
 	1    3700 6750
@@
 P 4200 6750
 F 0 "C2" H 4108 6704 50  0000 R CNN
-F 1 "C_Small" H 4108 6795 50  0000 R CNN
-F 2 "" H 4200 6750 50  0001 C CNN
+F 1 "0.01uF" H 4108 6795 50  0000 R CNN
+F 2 "Capacitor_SMD:C_0805_2012Metric_Pad1.15x1.40mm_HandSolder" H 4200 6750 50  0001 C CNN
 F 3 "~" H 4200 6750 50  0001 C CNN
 	1    4200 6750
@@
 P 4650 6750
 F 0 "C3" H 4558 6704 50  0000 R CNN
-F 1 "C_Small" H 4558 6795 50  0000 R CNN
-F 2 "" H 4650 6750 50  0001 C CNN
+F 1 "0.01uF" H 4558 6795 50  0000 R CNN
+F 2 "Capacitor_SMD:C_0805_2012Metric_Pad1.15x1.40mm_HandSolder" H 4650 6750 50  0001 C CNN
 F 3 "~" H 4650 6750 50  0001 C CNN
 	1    4650 6750
@@
 F 0 "J1" H 3220 3525 50  0000 C CNN
 F 1 "T_Admisión" H 3220 3616 50  0000 C CNN
-F 2 "" H 3300 3850 50  0001 C CNN
+F 2 "TerminalBlock:TerminalBlock_bornier-2_P5.08mm" H 3300 3850 50  0001 C CNN
 F 3 "~" H 3300 3850 50  0001 C CNN
 	1    3300 3850
@@
 F 0 "J2" H 3270 4325 50  0000 C CNN
 F 1 "T_Escape" H 3270 4416 50  0000 C CNN
-F 2 "" H 3350 4650 50  0001 C CNN
+F 2 "TerminalBlock:TerminalBlock_bornier-2_P5.08mm" H 3350 4650 50  0001 C CNN
 F 3 "~" H 3350 4650 50  0001 C CNN
 	1    3350 4650
@@
 F 0 "J3" H 3320 5125 50  0000 C CNN
 F 1 "T_Aceite" H 3320 5216 50  0000 C CNN
-F 2 "" H 3400 5450 50  0001 C CNN
+F 2 "TerminalBlock:TerminalBlock_bornier-2_P5.08mm" H 3400 5450 50  0001 C CNN
 F 3 "~" H 3400 5450 50  0001 C CNN
 	1    3400 5450
@@
 F 0 "U1" H 4450 4125 50  0000 C CNN
 F 1 "MAX31855" H 4450 4034 50  0000 C CNN
-F 2 "" H 4450 3750 50  0001 C CNN
+F 2 "Package_SO:SOIC-8_3.9x4.9mm_P1.27mm" H 4450 3750 50  0001 C CNN
 F 3 "" H 4450 3750 50  0001 C CNN
 	1    4450 3750
@@
 F 0 "U3" H 4450 5725 50  0000 C CNN
 F 1 "MAX31855" H 4450 5634 50  0000 C CNN
-F 2 "" H 4450 5350 50  0001 C CNN
+F 2 "Package_SO:SOIC-8_3.9x4.9mm_P1.27mm" H 4450 5350 50  0001 C CNN
 F 3 "" H 4450 5350 50  0001 C CNN
 	1    4450 5350
@@
 F 0 "U2" H 4450 4925 50  0000 C CNN
 F 1 "MAX31855" H 4450 4834 50  0000 C CNN
-F 2 "" H 4450 4550 50  0001 C CNN
+F 2 "Package_SO:SOIC-8_3.9x4.9mm_P1.27mm" H 4450 4550 50  0001 C CNN
 F 3 "" H 4450 4550 50  0001 C CNN
 	1    4450 4550

Commit message: Se cambio pack de 7805 y de 9044
Connections:
- wire segments 43 -> 47
Changed lines of the file:
@@
 	3700 6850 3700 6950
 Wire Wire Line
-	3700 6950 4650 6950
-Wire Wire Line
-	4650 6950 4650 6850
-Wire Wire Line
-	4200 7050 4200 6850
+	3700 6950 4200 6950
 $Comp
 L power:+3V3 #PWR013
@@
 	3700 6650 3700 6550
 Wire Wire Line
-	3700 6550 4650 6550
-Wire Wire Line
 	4650 6550 4650 6650
 Wire Wire Line
-	4200 6650 4200 6500
+	4200 6650 4200 6550
 Wire Wire Line
 	4800 3700 4850 3700
@@
 Wire Wire Line
 	3500 3750 4100 3750
+Wire Wire Line
+	4650 6550 4200 6550
+Connection ~ 4200 6550
+Wire Wire Line
+	4200 6550 4200 6500
+Wire Wire Line
+	3700 6550 4200 6550
+Wire Wire Line
+	4200 6850 4200 6950
+Connection ~ 4200 6950
+Wire Wire Line
+	4200 6950 4650 6950
+Wire Wire Line
+	4650 6850 4650 6950
+Wire Wire Line
+	4200 6950 4200 7050
 $EndSCHEMATC
