File: edu-ciaa.sch (KiCad schematic (older format))
At the start: 1 part

Commit message: Correccion de errores y se designaron huellas a casi todos los componentes
Other:
- note added: "Conectores EDU-CIAA"
- note added: "EDU-CIAA Conector A\n"
- note added: "EDU-CIAA Conector B"

Commit message: Ubicación de componentes y algo de ruteado
Changed lines of the file:
@@
 NoConn ~ 3350 3100
 NoConn ~ 3350 3200
-NoConn ~ 3350 3400
 NoConn ~ 3350 3700
 NoConn ~ 3350 3800
@@
 Text HLabel 4650 6800 2    50   Output ~ 0
 SCK
-Text HLabel 4650 6900 2    50   Output ~ 0
+Text HLabel 4650 7100 2    50   Output ~ 0
 ADM_CS
 Text HLabel 4650 7000 2    50   Output ~ 0
 ESC_CS
-Text HLabel 4650 7100 2    50   Output ~ 0
+Text HLabel 4650 6900 2    50   Output ~ 0
 ACT_CS
 Text HLabel 3300 4100 0    50   Input ~ 0
@@
 Text HLabel 4650 7400 2    50   Input ~ 0
 RPM_PULSE_I
-Text HLabel 3300 3600 0    50   Input ~ 0
+Text HLabel 3300 3400 0    50   Input ~ 0
 PRES_IN
 Text HLabel 3300 3500 0    50   Input ~ 0
@@
 	3300 3500 3350 3500
 Wire Wire Line
-	3300 3600 3350 3600
-Wire Wire Line
 	2850 3350 2850 3300
 Wire Wire Line
@@
 Text Notes 2550 2250 0    50   ~ 0
 Conectores EDU-CIAA
+Wire Wire Line
+	3300 3400 3350 3400
+NoConn ~ 3350 3600
 $EndSCHEMATC

Commit message: Se cambio pack de 7805 y de 9044
Connections:
- wire segments 78 -> 76
- no-connect marks 37 -> 38
Changed lines of the file:
@@
 $EndDescr
-$Comp
-L basico-rescue:+3.3V #PWR?
-U 1 1 61C156CC
-P 3150 2800
-AR Path="/61C156CC" Ref="#PWR?"  Part="1"
-AR Path="/61C15501/61C156CC" Ref="#PWR0101"  Part="1"
-F 0 "#PWR0101" H 3150 2760 30  0001 C CNN
-F 1 "+3.3V" H 3150 2910 30  0000 C CNN
-F 2 "" H 3150 2800 60  0000 C CNN
-F 3 "" H 3150 2800 60  0000 C CNN
-	1    3150 2800
-	1    0    0    -1
-$EndComp
 $Comp
 L basico-rescue:+5V #PWR?
@@
 	4750 3000 4750 2850
 Wire Wire Line
-	3150 2800 3150 3000
-Wire Wire Line
-	3150 3000 3350 3000
-Wire Wire Line
 	4550 5900 4750 5900
 Wire Wire Line
@@
 	3300 3400 3350 3400
 NoConn ~ 3350 3600
+NoConn ~ 3350 3000
 $EndSCHEMATC

Commit message: Ruteado de circuito de medicion de bateria
Connections:
- net labels added: V_BATT_IN
- wire segments 76 -> 77
- no-connect marks 38 -> 37
Changed lines of the file:
@@
 L basico-rescue:GND #PWR0113
 U 1 1 61C508C2
-P 2850 3350
-F 0 "#PWR0113" H 2850 3100 50  0001 C CNN
-F 1 "GND" H 2855 3177 50  0000 C CNN
-F 2 "" H 2850 3350 50  0000 C CNN
-F 3 "" H 2850 3350 50  0000 C CNN
-	1    2850 3350
+P 2850 3700
+F 0 "#PWR0113" H 2850 3450 50  0001 C CNN
+F 1 "GND" H 2855 3527 50  0000 C CNN
+F 2 "" H 2850 3700 50  0000 C CNN
+F 3 "" H 2850 3700 50  0000 C CNN
+	1    2850 3700
 	1    0    0    -1
 $EndComp
@@
 	3300 3500 3350 3500
 Wire Wire Line
-	2850 3350 2850 3300
-Wire Wire Line
 	2850 3300 3350 3300
 Wire Wire Line
@@
 Wire Wire Line
 	3300 3400 3350 3400
-NoConn ~ 3350 3600
 NoConn ~ 3350 3000
+Text HLabel 3300 3600 0    50   Input ~ 0
+V_BATT_IN
+Wire Wire Line
+	3300 3600 3350 3600
+Wire Wire Line
+	2850 3300 2850 3700
 $EndSCHEMATC
