File: ice-adq.sch (KiCad schematic (older format))
At the start: 4 parts

Commit message: Terminado el esquemático para los amplificadores de termocuplas
Parts:
- removed U? (x3): MAX31855KASA, Package_SO:SOIC-8_3.9x4.9mm_P1.27mm, symbol Sensor_Temperature:MAX31855KASA
Changed lines of the file:
@@
 EESchema Schematic File Version 4
-EELAYER 30 0
+LIBS:ice-adq-cache
+EELAYER 26 0
 EELAYER END
 $Descr A4 11693 8268
 encoding utf-8
-Sheet 1 1
+Sheet 1 5
 Title "Poncho Básico (Editar y colocar el nombre final)"
 Date "2016-08-07"
@@
 Wire Wire Line
 	3250 1450 3700 1450
-$Comp
-L Sensor_Temperature:MAX31855KASA U?
-U 1 1 5FF5C03E
-P 7500 3850
-F 0 "U?" H 7500 4431 50  0000 C CNN
-F 1 "MAX31855KASA" H 7500 4340 50  0000 C CNN
-F 2 "Package_SO:SOIC-8_3.9x4.9mm_P1.27mm" H 8500 3500 50  0001 C CIN
-F 3 "http://datasheets.maximintegrated.com/en/ds/MAX31855.pdf" H 7500 3850 50  0001 C CNN
-	1    7500 3850
-	1    0    0    -1
-$EndComp
-$Comp
-L Sensor_Temperature:MAX31855KASA U?
-U 1 1 5FF5CC5C
-P 8850 3850
-F 0 "U?" H 8850 4431 50  0000 C CNN
-F 1 "MAX31855KASA" H 8850 4340 50  0000 C CNN
-F 2 "Package_SO:SOIC-8_3.9x4.9mm_P1.27mm" H 9850 3500 50  0001 C CIN
-F 3 "http://datasheets.maximintegrated.com/en/ds/MAX31855.pdf" H 8850 3850 50  0001 C CNN
-	1    8850 3850
-	1    0    0    -1
-$EndComp
-$Comp
-L Sensor_Temperature:MAX31855KASA U?
-U 1 1 5FF5D74D
-P 6250 3850
-F 0 "U?" H 6250 4431 50  0000 C CNN
-F 1 "MAX31855KASA" H 6250 4340 50  0000 C CNN
-F 2 "Package_SO:SOIC-8_3.9x4.9mm_P1.27mm" H 7250 3500 50  0001 C CIN
-F 3 "http://datasheets.maximintegrated.com/en/ds/MAX31855.pdf" H 6250 3850 50  0001 C CNN
-	1    6250 3850
-	1    0    0    -1
-$EndComp
+$Sheet
+S 4700 1750 1100 900
+U 5FFF8913
+F0 "termocuplas" 50
+F1 "termocuplas.sch" 50
+$EndSheet
+$Sheet
+S 4750 3000 1000 900
+U 5FFFA450
+F0 "oxigeno" 50
+F1 "oxigeno.sch" 50
+$EndSheet
+$Sheet
+S 6300 2950 1050 1050
+U 5FFFA455
+F0 "rpm" 50
+F1 "rpm.sch" 50
+$EndSheet
+$Sheet
+S 4700 4350 950  900
+U 5FFFA45A
+F0 "presion" 50
+F1 "presion.sch" 50
+$EndSheet
+$Sheet
+S 6350 4400 1000 900
+U 5FFFA45F
+F0 "comunicaciones" 50
+F1 "comunicaciones.sch" 50
+$EndSheet
 $EndSCHEMATC

Commit message: Primer rev esquematicos RPM y comunicaciones
Changed lines of the file:
@@
 $Descr A4 11693 8268
 encoding utf-8
-Sheet 1 5
+Sheet 1 6
 Title "Poncho Básico (Editar y colocar el nombre final)"
 Date "2016-08-07"
 Rev "1.0"
-Comp "Proyecto CIAA - COMPUTADORA INDUSTRIAL ABIERTA ARGENTINA"
-Comment1 "https://github.com/ciaa/Ponchos/tree/master/Basico/doc"
-Comment2 "Autores y Licencia del modelo (Diego Brengi - UNLaM)"
+Comp "Autor: Ignacio Moya"
+Comment1 "Autor: Ignacio Moya"
+Comment2 "Especialización en Sistemas Embebidos 2021 - FIUBA"
 Comment3 "Autor del poncho (COMPLETAR NOMBRE Y APELLIDO). Ver directorio \"doc\""
 Comment4 ""
@@
 	3250 1450 3700 1450
 $Sheet
-S 4700 1750 1100 900
+S 4700 1750 850  600
 U 5FFF8913
 F0 "termocuplas" 50
 F1 "termocuplas.sch" 50
+F2 "SO" O L 4700 1850 50
+F3 "SCK" I L 4700 1950 50
+F4 "ADM_CS" I L 4700 2050 50
+F5 "ESC_CS" I L 4700 2150 50
+F6 "ACT_CS" I L 4700 2250 50
 $EndSheet
 $Sheet
-S 4750 3000 1000 900
+S 4700 5450 1000 900
 U 5FFFA450
 F0 "oxigeno" 50
@@
 $EndSheet
 $Sheet
-S 6300 2950 1050 1050
+S 4700 3200 1000 400
 U 5FFFA455
 F0 "rpm" 50
 F1 "rpm.sch" 50
+F2 "RPM_PULSE" I L 4700 3400 50
 $EndSheet
 $Sheet
-S 4700 4350 950  900
+S 4700 4400 950  900
 U 5FFFA45A
 F0 "presion" 50
@@
 $EndSheet
 $Sheet
-S 6350 4400 1000 900
+S 4700 2550 950  500
 U 5FFFA45F
 F0 "comunicaciones" 50
 F1 "comunicaciones.sch" 50
+F2 "BT_TX" I L 4700 2700 50
+F3 "BT_RX" I L 4700 2800 50
+F4 "BT_STATE" I L 4700 2900 50
 $EndSheet
 $EndSCHEMATC

Commit message: Esquematicos mayormente terminados, falta sub-hoja edu ciaa, fuentes de alimentacion y poner valores a los componentes
Changed lines of the file:
@@
 Rev "1.0"
 Comp "Autor: Ignacio Moya"
-Comment1 "Autor: Ignacio Moya"
-Comment2 "Especialización en Sistemas Embebidos 2021 - FIUBA"
-Comment3 "Autor del poncho (COMPLETAR NOMBRE Y APELLIDO). Ver directorio \"doc\""
+Comment1 "Especialización en Sistemas Embebidos 2021 - FIUBA"
+Comment2 ""
+Comment3 ""
 Comment4 ""
 $EndDescr
@@
 	3250 1450 3700 1450
 $Sheet
-S 4700 1750 850  600
+S 4700 1750 950  600
 U 5FFF8913
 F0 "termocuplas" 50
@@
 $EndSheet
 $Sheet
-S 4700 3200 1000 400
+S 4700 3200 950  400
 U 5FFFA455
 F0 "rpm" 50
@@
 $EndSheet
 $Sheet
-S 4700 4400 950  900
+S 4700 3800 950  300
 U 5FFFA45A
 F0 "presion" 50
 F1 "presion.sch" 50
+F2 "PRES_OUT" I L 4700 3950 50
 $EndSheet
 $Sheet

Commit message: Se agrego esquematico de fuentes y se corrigieron errores de ERC
Parts:
- removed XA101: Conn_Poncho2P_2x_20x2, footprint:Conn_Poncho_SinBorde, symbol basico-rescue:Conn_Poncho2P_2x_20x2
Connections:
- net labels removed: +3.3V, +3.3VP, +5V, +5VP, GND, GNDA, GNDD
- wire segments 76 -> 33
- no-connect marks 48 -> 0
Other:
- note removed: "Borrar si no se quiere \nconexiones entre ambos \nconectores"

Commit message: Correccion de errores y se designaron huellas a casi todos los componentes
Other:
- note removed: "Este diseño puede copiarse para iniciar un poncho simple. \n1) Copiar toda la carpeta "Basico" , renombrando \n la misma al nombre del poncho.\n2) Renombrar los archivos "basico.xxx" manteniendo \n las extensiones pero cambiando a un nombre \n descriptivo del poncho. Evitar acentos, espacios y \n caracteres ascii esxtendidos."
Changed lines of the file:
@@
 Sheet 1 8
 Title "Poncho adquisidor de datos para motor de combustión interna"
-Date "2021-12-18"
+Date "2021-12-19"
 Rev "1.0"
 Comp "Autor: Ignacio Moya"
@@
 	1    0    0    -1
 $EndComp
-Text Notes 7500 1850 0    79   Italic 16
-Este diseño puede copiarse para iniciar un poncho simple. \n1) Copiar toda la carpeta "Basico" , renombrando \n   la misma al nombre del poncho.\n2) Renombrar los archivos "basico.xxx" manteniendo \n    las extensiones pero cambiando a un nombre \n    descriptivo del poncho. Evitar acentos, espacios y \n    caracteres ascii esxtendidos.
 Text Notes 7550 800  0    118  ~ 24
 http://www.proyecto-ciaa.com.ar/
@@
 Luego de abrir el nuevo proyecto:\n1)Editar datos del rótulo.\n2)Editar los archivos del subdirectorio "doc".\n2.1) Agregarse en el archivo de licencia.\n2.2) Colocar info mínima del Poncho en el LEEME.txt\n2.3) Colocar info mínima en el CAMBIOS.txt
 $Sheet
-S 4700 1750 950  600
+S 7100 1900 950  600
 U 5FFF8913
 F0 "termocuplas" 50
 F1 "termocuplas.sch" 50
-F2 "SO" O L 4700 1850 50
-F3 "SCK" I L 4700 1950 50
-F4 "ADM_CS" I L 4700 2050 50
-F5 "ESC_CS" I L 4700 2150 50
-F6 "ACT_CS" I L 4700 2250 50
+F2 "SO" O L 7100 2000 50
+F3 "SCK" I L 7100 2100 50
+F4 "ADM_CS" I L 7100 2200 50
+F5 "ESC_CS" I L 7100 2300 50
+F6 "ACT_CS" I L 7100 2400 50
 $EndSheet
 $Sheet
-S 4700 4350 950  300
+S 7100 4500 950  300
 U 5FFFA450
 F0 "oxigeno" 50
 F1 "oxigeno.sch" 50
-F2 "O2_OUT" I L 4700 4500 50
+F2 "O2_OUT" I L 7100 4650 50
 $EndSheet
 $Sheet
-S 4700 3250 950  400
+S 7100 3400 950  400
 U 5FFFA455
 F0 "rpm" 50
 F1 "rpm.sch" 50
-F2 "RPM_PULSE" O L 4700 3450 50
+F2 "RPM_PULSE" O L 7100 3600 50
 $EndSheet
 $Sheet
-S 4700 3850 950  300
+S 7100 4000 950  300
 U 5FFFA45A
 F0 "presion" 50
 F1 "presion.sch" 50
-F2 "PRES_OUT" I L 4700 4000 50
+F2 "PRES_OUT" I L 7100 4150 50
 $EndSheet
 $Sheet
-S 4700 2550 950  500
+S 7100 2700 950  500
 U 5FFFA45F
 F0 "comunicaciones" 50
 F1 "comunicaciones.sch" 50
-F2 "BT_TX" O L 4700 2700 50
-F3 "BT_STATE" O L 4700 2900 50
-F4 "BT_RX" I L 4700 2800 50
+F2 "BT_TX" O L 7100 2850 50
+F3 "BT_STATE" O L 7100 3050 50
+F4 "BT_RX" I L 7100 2950 50
 $EndSheet
 $Sheet
-S 1650 4100 700  500
+S 4050 4250 700  500
 U 61C1A3CD
 F0 "fuentes" 50
@@
 $EndSheet
 $Sheet
-S 1550 2200 850  1650
+S 3950 2350 850  1650
 U 61C15501
 F0 "edu-ciaa" 50
 F1 "edu-ciaa.sch" 50
-F2 "SO" I R 2400 2300 50
-F3 "SCK" O R 2400 2400 50
-F4 "ADM_CS" O R 2400 2500 50
-F5 "ESC_CS" O R 2400 2600 50
-F6 "ACT_CS" O R 2400 2700 50
-F7 "BT_TX" I R 2400 2900 50
-F8 "BT_RX" O R 2400 3000 50
-F9 "BT_STATE" I R 2400 3100 50
-F10 "RPM_PULSE_I" I R 2400 3300 50
-F11 "PRES_IN" I R 2400 3500 50
-F12 "O2_IN" I R 2400 3700 50
+F2 "SO" I R 4800 2450 50
+F3 "SCK" O R 4800 2550 50
+F4 "ADM_CS" O R 4800 2650 50
+F5 "ESC_CS" O R 4800 2750 50
+F6 "ACT_CS" O R 4800 2850 50
+F7 "BT_TX" I R 4800 3050 50
+F8 "BT_RX" O R 4800 3150 50
+F9 "BT_STATE" I R 4800 3250 50
+F10 "RPM_PULSE_I" I R 4800 3450 50
+F11 "PRES_IN" I R 4800 3650 50
+F12 "O2_IN" I R 4800 3850 50
 $EndSheet
 Wire Wire Line
-	3550 2300 3550 1850
+	5950 2450 5950 2000
 Wire Wire Line
-	3550 1850 4700 1850
+	5950 2000 7100 2000
 Wire Wire Line
-	4700 1950 3650 1950
+	7100 2100 6050 2100
 Wire Wire Line
-	3650 1950 3650 2400
+	6050 2100 6050 2550
 Wire Wire Line
-	3650 2400 2400 2400
+	6050 2550 4800 2550
 Wire Wire Line
-	2400 2500 3750 2500
+	4800 2650 6150 2650
 Wire Wire Line
-	3750 2500 3750 2050
+	6150 2650 6150 2200
 Wire Wire Line
-	3750 2050 4700 2050
+	6150 2200 7100 2200
 Wire Wire Line
-	4700 2150 3850 2150
+	7100 2300 6250 2300
 Wire Wire Line
-	3850 2150 3850 2600
+	6250 2300 6250 2750
 Wire Wire Line
-	3850 2600 2400 2600
+	6250 2750 4800 2750
 Wire Wire Line
-	2400 2700 3950 2700
+	4800 2850 6350 2850
 Wire Wire Line
-	3950 2700 3950 2250
+	6350 2850 6350 2400
 Wire Wire Line
-	3950 2250 4700 2250
+	6350 2400 7100 2400
 Wire Wire Line
-	2400 2300 3550 2300
+	4800 2450 5950 2450
 Wire Wire Line
-	2400 2900 4200 2900
+	4800 3050 6600 3050
 Wire Wire Line
-	4200 2900 4200 2700
+	6600 3050 6600 2850
 Wire Wire Line
-	4200 2700 4700 2700
+	6600 2850 7100 2850
 Wire Wire Line
-	4700 2800 4300 2800
+	7100 2950 6700 2950
 Wire Wire Line
-	4300 2800 4300 3000
+	6700 2950 6700 3150
 Wire Wire Line
-	4300 3000 2400 3000
+	6700 3150 4800 3150
 Wire Wire Line
-	4400 3100 4400 2900
+	6800 3250 6800 3050
 Wire Wire Line
-	4400 2900 4700 2900
+	6800 3050 7100 3050
 Wire Wire Line
-	2400 3100 4400 3100
+	4800 3250 6800 3250
 Wire Wire Line
-	2400 3300 4400 3300
+	4800 3450 6800 3450
 Wire Wire Line
-	4400 3300 4400 3450
+	6800 3450 6800 3600
 Wire Wire Line
-	4400 3450 4700 3450
+	6800 3600 7100 3600
 Wire Wire Line
-	4700 4000 4100 4000
+	7100 4150 6500 4150
 Wire Wire Line
-	4100 4000 4100 3500
+	6500 4150 6500 3650
 Wire Wire Line
-	4100 3500 2400 3500
+	6500 3650 4800 3650
 Wire Wire Line
-	2400 3700 3700 3700
+	4800 3850 6100 3850
 Wire Wire Line
-	3700 3700 3700 4500
+	6100 3850 6100 4650
 Wire Wire Line
-	3700 4500 4700 4500
+	6100 4650 7100 4650
 $EndSCHEMATC

Commit message: Ruteado de circuito de medicion de bateria
Connections:
- wire segments 33 -> 12
Changed lines of the file:
@@
 Luego de abrir el nuevo proyecto:\n1)Editar datos del rótulo.\n2)Editar los archivos del subdirectorio "doc".\n2.1) Agregarse en el archivo de licencia.\n2.2) Colocar info mínima del Poncho en el LEEME.txt\n2.3) Colocar info mínima en el CAMBIOS.txt
 $Sheet
-S 7100 1900 950  600
+S 7700 3000 950  600
 U 5FFF8913
 F0 "termocuplas" 50
 F1 "termocuplas.sch" 50
-F2 "SO" O L 7100 2000 50
-F3 "SCK" I L 7100 2100 50
-F4 "ADM_CS" I L 7100 2200 50
-F5 "ESC_CS" I L 7100 2300 50
-F6 "ACT_CS" I L 7100 2400 50
+F2 "SO" O L 7700 3100 50
+F3 "SCK" I L 7700 3200 50
+F4 "ADM_CS" I L 7700 3300 50
+F5 "ESC_CS" I L 7700 3400 50
+F6 "ACT_CS" I L 7700 3500 50
 $EndSheet
 $Sheet
-S 7100 4500 950  300
+S 3850 3750 950  300
 U 5FFFA450
 F0 "oxigeno" 50
 F1 "oxigeno.sch" 50
-F2 "O2_OUT" I L 7100 4650 50
+F2 "O2_OUT" I R 4800 3900 50
 $EndSheet
 $Sheet
-S 7100 3400 950  400
+S 3850 2850 950  300
 U 5FFFA455
 F0 "rpm" 50
 F1 "rpm.sch" 50
-F2 "RPM_PULSE" O L 7100 3600 50
+F2 "RPM_PULSE" O R 4800 3000 50
 $EndSheet
 $Sheet
-S 7100 4000 950  300
+S 3850 3300 950  300
 U 5FFFA45A
 F0 "presion" 50
 F1 "presion.sch" 50
-F2 "PRES_OUT" I L 7100 4150 50
+F2 "PRES_OUT" I R 4800 3450 50
 $EndSheet
 $Sheet
-S 7100 2700 950  500
+S 7700 3800 950  500
 U 5FFFA45F
 F0 "comunicaciones" 50
 F1 "comunicaciones.sch" 50
-F2 "BT_TX" O L 7100 2850 50
-F3 "BT_STATE" O L 7100 3050 50
-F4 "BT_RX" I L 7100 2950 50
+F2 "BT_TX" O L 7700 3950 50
+F3 "BT_STATE" O L 7700 4150 50
+F4 "BT_RX" I L 7700 4050 50
 $EndSheet
 $Sheet
-S 4050 4250 700  500
+S 3850 4200 950  300
 U 61C1A3CD
 F0 "fuentes" 50
 F1 "fuentes.sch" 50
+F2 "V_BATT_OUT" O R 4800 4350 50
 $EndSheet
 $Sheet
-S 3950 2350 850  1650
+S 5600 2850 1150 1650
 U 61C15501
 F0 "edu-ciaa" 50
 F1 "edu-ciaa.sch" 50
-F2 "SO" I R 4800 2450 50
-F3 "SCK" O R 4800 2550 50
-F4 "ADM_CS" O R 4800 2650 50
-F5 "ESC_CS" O R 4800 2750 50
-F6 "ACT_CS" O R 4800 2850 50
-F7 "BT_TX" I R 4800 3050 50
-F8 "BT_RX" O R 4800 3150 50
-F9 "BT_STATE" I R 4800 3250 50
-F10 "RPM_PULSE_I" I R 4800 3450 50
-F11 "PRES_IN" I R 4800 3650 50
-F12 "O2_IN" I R 4800 3850 50
+F2 "SO" I R 6750 3100 50
+F3 "SCK" O R 6750 3200 50
+F4 "ADM_CS" O R 6750 3300 50
+F5 "ESC_CS" O R 6750 3400 50
+F6 "ACT_CS" O R 6750 3500 50
+F7 "BT_TX" I R 6750 3950 50
+F8 "BT_RX" O R 6750 4050 50
+F9 "BT_STATE" I R 6750 4150 50
+F10 "RPM_PULSE_I" I L 5600 3000 50
+F11 "PRES_IN" I L 5600 3450 50
+F12 "O2_IN" I L 5600 3900 50
+F13 "V_BATT_IN" I L 5600 4350 50
 $EndSheet
 Wire Wire Line
-	5950 2450 5950 2000
+	4800 4350 5600 4350
 Wire Wire Line
-	5950 2000 7100 2000
+	4800 3900 5600 3900
 Wire Wire Line
-	7100 2100 6050 2100
+	4800 3450 5600 3450
 Wire Wire Line
-	6050 2100 6050 2550
+	4800 3000 5600 3000
 Wire Wire Line
-	6050 2550 4800 2550
+	6750 3100 7700 3100
 Wire Wire Line
-	4800 2650 6150 2650
+	7700 3200 6750 3200
 Wire Wire Line
-	6150 2650 6150 2200
+	6750 3300 7700 3300
 Wire Wire Line
-	6150 2200 7100 2200
+	7700 3400 6750 3400
 Wire Wire Line
-	7100 2300 6250 2300
+	6750 3500 7700 3500
 Wire Wire Line
-	6250 2300 6250 2750
+	7700 3950 6750 3950
 Wire Wire Line
-	6250 2750 4800 2750
+	6750 4050 7700 4050
 Wire Wire Line
-	4800 2850 6350 2850
-Wire Wire Line
-	6350 2850 6350 2400
-Wire Wire Line
-	6350 2400 7100 2400
-Wire Wire Line
-	4800 2450 5950 2450
-Wire Wire Line
-	4800 3050 6600 3050
-Wire Wire Line
-	6600 3050 6600 2850
-Wire Wire Line
-	6600 2850 7100 2850
-Wire Wire Line
-	7100 2950 6700 2950
-Wire Wire Line
-	6700 2950 6700 3150
-Wire Wire Line
-	6700 3150 4800 3150
-Wire Wire Line
-	6800 3250 6800 3050
-Wire Wire Line
-	6800 3050 7100 3050
-Wire Wire Line
-	4800 3250 6800 3250
-Wire Wire Line
-	4800 3450 6800 3450
-Wire Wire Line
-	6800 3450 6800 3600
-Wire Wire Line
-	6800 3600 7100 3600
-Wire Wire Line
-	7100 4150 6500 4150
-Wire Wire Line
-	6500 4150 6500 3650
-Wire Wire Line
-	6500 3650 4800 3650
-Wire Wire Line
-	4800 3850 6100 3850
-Wire Wire Line
-	6100 3850 6100 4650
-Wire Wire Line
-	6100 4650 7100 4650
+	7700 4150 6750 4150
 $EndSCHEMATC
