File: comunicaciones.sch (KiCad schematic (older format))
At the start: 0 parts

Commit message: Primer rev esquematicos RPM y comunicaciones
Parts:
- added R?: hm10, symbol hm10:hm10
Connections:
- net labels added: +3.3V, BT_RX, BT_STATE, BT_TX, GND
- wire segments 0 -> 7
Changed lines of the file:
@@
 $Descr A4 11693 8268
 encoding utf-8
-Sheet 1 1
+Sheet 6 6
 Title ""
 Date ""
 Rev ""
-Comp ""
-Comment1 ""
-Comment2 ""
+Comp "Autor: Ignacio Moya"
+Comment1 "Autor: Ignacio Moya"
+Comment2 "Especialización en Sistemas Embebidos 2021 - FIUBA"
 Comment3 ""
 Comment4 ""
 $EndDescr
+$Comp
+L hm10:hm10 R?
+U 1 1 61B55EEA
+P 7050 3950
+F 0 "R?" H 7328 3996 50  0000 L CNN
+F 1 "hm10" H 7328 3905 50  0000 L CNN
+F 2 "" V 7100 3700 50  0001 L CNN
+F 3 "" H 7000 3900 50  0001 C CNN
+	1    7050 3950
+	1    0    0    -1
+$EndComp
+$Comp
+L power:+3.3V #PWR?
+U 1 1 61B55F54
+P 6600 3600
+F 0 "#PWR?" H 6600 3450 50  0001 C CNN
+F 1 "+3.3V" H 6615 3773 50  0000 C CNN
+F 2 "" H 6600 3600 50  0001 C CNN
+F 3 "" H 6600 3600 50  0001 C CNN
+	1    6600 3600
+	1    0    0    -1
+$EndComp
+$Comp
+L basico-rescue:GND #PWR?
+U 1 1 61B55F96
+P 6600 4300
+F 0 "#PWR?" H 6600 4050 50  0001 C CNN
+F 1 "GND" H 6605 4127 50  0000 C CNN
+F 2 "" H 6600 4300 50  0000 C CNN
+F 3 "" H 6600 4300 50  0000 C CNN
+	1    6600 4300
+	1    0    0    -1
+$EndComp
+Wire Wire Line
+	6600 4300 6600 4200
+Wire Wire Line
+	6600 4200 6650 4200
+Wire Wire Line
+	6650 3700 6600 3700
+Wire Wire Line
+	6600 3700 6600 3600
+Wire Wire Line
+	6250 3850 6650 3850
+Wire Wire Line
+	6250 3950 6650 3950
+Wire Wire Line
+	6250 4050 6650 4050
+Text HLabel 6250 3850 0    50   Input ~ 0
+BT_TX
+Text HLabel 6250 3950 0    50   Input ~ 0
+BT_RX
+Text HLabel 6250 4050 0    50   Input ~ 0
+BT_STATE
 $EndSCHEMATC

Commit message: Esquematicos mayormente terminados, falta sub-hoja edu ciaa, fuentes de alimentacion y poner valores a los componentes
Parts:
- added C?: C_Small, symbol Device:C_Small
- gave numbers to parts that had none: 1
Connections:
- wire segments 7 -> 11
Other:
- note added: "Módulo Bluetooth HM-10"
Changed lines of the file:
@@
 EELAYER 26 0
 EELAYER END
-$Descr A4 11693 8268
+$Descr A4 8268 11693 portrait
 encoding utf-8
 Sheet 6 6
@@
 Rev ""
 Comp "Autor: Ignacio Moya"
-Comment1 "Autor: Ignacio Moya"
-Comment2 "Especialización en Sistemas Embebidos 2021 - FIUBA"
+Comment1 "Especialización en Sistemas Embebidos 2021 - FIUBA"
+Comment2 ""
 Comment3 ""
 Comment4 ""
 $EndDescr
 $Comp
-L hm10:hm10 R?
+L hm10:hm10 U?
 U 1 1 61B55EEA
-P 7050 3950
-F 0 "R?" H 7328 3996 50  0000 L CNN
-F 1 "hm10" H 7328 3905 50  0000 L CNN
-F 2 "" V 7100 3700 50  0001 L CNN
-F 3 "" H 7000 3900 50  0001 C CNN
-	1    7050 3950
+P 4600 5900
+F 0 "U?" H 4878 5946 50  0000 L CNN
+F 1 "hm10" H 4878 5855 50  0000 L CNN
+F 2 "" V 4650 5650 50  0001 L CNN
+F 3 "" H 4550 5850 50  0001 C CNN
+	1    4600 5900
 	1    0    0    -1
 $EndComp
@@
 L power:+3.3V #PWR?
 U 1 1 61B55F54
-P 6600 3600
-F 0 "#PWR?" H 6600 3450 50  0001 C CNN
-F 1 "+3.3V" H 6615 3773 50  0000 C CNN
-F 2 "" H 6600 3600 50  0001 C CNN
-F 3 "" H 6600 3600 50  0001 C CNN
-	1    6600 3600
+P 4150 5300
+F 0 "#PWR?" H 4150 5150 50  0001 C CNN
+F 1 "+3.3V" H 4165 5473 50  0000 C CNN
+F 2 "" H 4150 5300 50  0001 C CNN
+F 3 "" H 4150 5300 50  0001 C CNN
+	1    4150 5300
 	1    0    0    -1
 $EndComp
@@
 L basico-rescue:GND #PWR?
 U 1 1 61B55F96
-P 6600 4300
-F 0 "#PWR?" H 6600 4050 50  0001 C CNN
-F 1 "GND" H 6605 4127 50  0000 C CNN
-F 2 "" H 6600 4300 50  0000 C CNN
-F 3 "" H 6600 4300 50  0000 C CNN
-	1    6600 4300
+P 4150 6250
+F 0 "#PWR?" H 4150 6000 50  0001 C CNN
+F 1 "GND" H 4155 6077 50  0000 C CNN
+F 2 "" H 4150 6250 50  0000 C CNN
+F 3 "" H 4150 6250 50  0000 C CNN
+	1    4150 6250
 	1    0    0    -1
 $EndComp
 Wire Wire Line
-	6600 4300 6600 4200
+	4150 6250 4150 6150
 Wire Wire Line
-	6600 4200 6650 4200
+	4150 6150 4200 6150
 Wire Wire Line
-	6650 3700 6600 3700
+	4200 5650 4150 5650
 Wire Wire Line
-	6600 3700 6600 3600
+	3800 5800 4200 5800
 Wire Wire Line
-	6250 3850 6650 3850
+	3800 5900 4200 5900
 Wire Wire Line
-	6250 3950 6650 3950
+	3800 6000 4200 6000
+Text HLabel 3800 5800 0    50   Input ~ 0
+BT_TX
+Text HLabel 3800 5900 0    50   Input ~ 0
+BT_RX
+Text HLabel 3800 6000 0    50   Input ~ 0
+BT_STATE
+$Comp
+L Device:C_Small C?
+U 1 1 61BB32CB
+P 4000 5450
+F 0 "C?" V 3863 5450 50  0000 C CNN
+F 1 "C_Small" H 4092 5405 50  0001 L CNN
+F 2 "" H 4000 5450 50  0001 C CNN
+F 3 "~" H 4000 5450 50  0001 C CNN
+	1    4000 5450
+	0    1    1    0
+$EndComp
+$Comp
+L basico-rescue:GND #PWR?
+U 1 1 61BB3391
+P 3800 5500
+F 0 "#PWR?" H 3800 5250 50  0001 C CNN
+F 1 "GND" H 3805 5327 50  0000 C CNN
+F 2 "" H 3800 5500 50  0000 C CNN
+F 3 "" H 3800 5500 50  0000 C CNN
+	1    3800 5500
+	1    0    0    -1
+$EndComp
 Wire Wire Line
-	6250 4050 6650 4050
-Text HLabel 6250 3850 0    50   Input ~ 0
-BT_TX
-Text HLabel 6250 3950 0    50   Input ~ 0
-BT_RX
-Text HLabel 6250 4050 0    50   Input ~ 0
-BT_STATE
+	3800 5500 3800 5450
+Wire Wire Line
+	3800 5450 3900 5450
+Wire Wire Line
+	4100 5450 4150 5450
+Wire Wire Line
+	4150 5450 4150 5650
+Wire Wire Line
+	4150 5300 4150 5450
+Connection ~ 4150 5450
+Wire Notes Line
+	3100 4900 5400 4900
+Wire Notes Line
+	5400 4900 5400 6600
+Wire Notes Line
+	5400 6600 3100 6600
+Wire Notes Line
+	3100 6600 3100 4900
+Text Notes 3100 4850 0    50   ~ 0
+Módulo Bluetooth HM-10
 $EndSCHEMATC

Commit message: Se agrego esquematico de fuentes y se corrigieron errores de ERC
Parts:
- gave numbers to parts that had none: 2
Changed lines of the file:
@@
 $Descr A4 8268 11693 portrait
 encoding utf-8
-Sheet 6 6
+Sheet 6 8
 Title ""
-Date ""
-Rev ""
+Date "2021-12-18"
+Rev "1.0"
 Comp "Autor: Ignacio Moya"
 Comment1 "Especialización en Sistemas Embebidos 2021 - FIUBA"
@@
 $EndDescr
 $Comp
-L hm10:hm10 U?
+L hm10:hm10 U8
 U 1 1 61B55EEA
 P 4600 5900
-F 0 "U?" H 4878 5946 50  0000 L CNN
+F 0 "U8" H 4878 5946 50  0000 L CNN
 F 1 "hm10" H 4878 5855 50  0000 L CNN
 F 2 "" V 4650 5650 50  0001 L CNN
@@
 $EndComp
 $Comp
-L power:+3.3V #PWR?
+L power:+3.3V #PWR039
 U 1 1 61B55F54
 P 4150 5300
-F 0 "#PWR?" H 4150 5150 50  0001 C CNN
+F 0 "#PWR039" H 4150 5150 50  0001 C CNN
 F 1 "+3.3V" H 4165 5473 50  0000 C CNN
 F 2 "" H 4150 5300 50  0001 C CNN
@@
 $EndComp
 $Comp
-L basico-rescue:GND #PWR?
+L basico-rescue:GND #PWR040
 U 1 1 61B55F96
 P 4150 6250
-F 0 "#PWR?" H 4150 6000 50  0001 C CNN
+F 0 "#PWR040" H 4150 6000 50  0001 C CNN
 F 1 "GND" H 4155 6077 50  0000 C CNN
 F 2 "" H 4150 6250 50  0000 C CNN
@@
 Wire Wire Line
 	3800 6000 4200 6000
-Text HLabel 3800 5800 0    50   Input ~ 0
+Text HLabel 3800 5800 0    50   Output ~ 0
 BT_TX
 Text HLabel 3800 5900 0    50   Input ~ 0
 BT_RX
-Text HLabel 3800 6000 0    50   Input ~ 0
+Text HLabel 3800 6000 0    50   Output ~ 0
 BT_STATE
 $Comp
-L Device:C_Small C?
+L Device:C_Small C13
 U 1 1 61BB32CB
 P 4000 5450
-F 0 "C?" V 3863 5450 50  0000 C CNN
+F 0 "C13" V 3863 5450 50  0000 C CNN
 F 1 "C_Small" H 4092 5405 50  0001 L CNN
 F 2 "" H 4000 5450 50  0001 C CNN
@@
 $EndComp
 $Comp
-L basico-rescue:GND #PWR?
+L basico-rescue:GND #PWR038
 U 1 1 61BB3391
 P 3800 5500
-F 0 "#PWR?" H 3800 5250 50  0001 C CNN
+F 0 "#PWR038" H 3800 5250 50  0001 C CNN
 F 1 "GND" H 3805 5327 50  0000 C CNN
 F 2 "" H 3800 5500 50  0000 C CNN

Commit message: Correccion de errores y se designaron huellas a casi todos los componentes
Parts:
- C13: value C_Small -> 0.01uF; footprint (none) -> Capacitor_SMD:C_0805_2012Metric_Pad1.15x1.40mm_HandSolder
Changed lines of the file:
@@
 Sheet 6 8
 Title ""
-Date "2021-12-18"
+Date "2021-12-19"
 Rev "1.0"
 Comp "Autor: Ignacio Moya"
@@
 L power:+3.3V #PWR039
 U 1 1 61B55F54
-P 4150 5300
-F 0 "#PWR039" H 4150 5150 50  0001 C CNN
-F 1 "+3.3V" H 4165 5473 50  0000 C CNN
-F 2 "" H 4150 5300 50  0001 C CNN
-F 3 "" H 4150 5300 50  0001 C CNN
-	1    4150 5300
+P 4150 5200
+F 0 "#PWR039" H 4150 5050 50  0001 C CNN
+F 1 "+3.3V" H 4165 5373 50  0000 C CNN
+F 2 "" H 4150 5200 50  0001 C CNN
+F 3 "" H 4150 5200 50  0001 C CNN
+	1    4150 5200
 	1    0    0    -1
 $EndComp
@@
 U 1 1 61BB32CB
 P 4000 5450
-F 0 "C13" V 3863 5450 50  0000 C CNN
-F 1 "C_Small" H 4092 5405 50  0001 L CNN
-F 2 "" H 4000 5450 50  0001 C CNN
+F 0 "C13" V 3800 5450 50  0000 C CNN
+F 1 "0.01uF" V 3900 5300 50  0000 L CNN
+F 2 "Capacitor_SMD:C_0805_2012Metric_Pad1.15x1.40mm_HandSolder" H 4000 5450 50  0001 C CNN
 F 3 "~" H 4000 5450 50  0001 C CNN
 	1    4000 5450
@@
 Wire Wire Line
 	4150 5450 4150 5650
-Wire Wire Line
-	4150 5300 4150 5450
 Connection ~ 4150 5450
 Wire Notes Line
@@
 Text Notes 3100 4850 0    50   ~ 0
 Módulo Bluetooth HM-10
+Wire Wire Line
+	4150 5200 4150 5450
 $EndSCHEMATC

Commit message: Se agregaron modelos 3d faltantes
Parts:
- U8: footprint (none) -> Connector_PinHeader_2.54mm:PinHeader_1x06_P2.54mm_Vertical
Changed lines of the file:
@@
 F 0 "U8" H 4878 5946 50  0000 L CNN
 F 1 "hm10" H 4878 5855 50  0000 L CNN
-F 2 "" V 4650 5650 50  0001 L CNN
+F 2 "Connector_PinHeader_2.54mm:PinHeader_1x06_P2.54mm_Vertical" V 4650 5650 50  0001 L CNN
 F 3 "" H 4550 5850 50  0001 C CNN
 	1    4600 5900

Commit message: Comitee cambios que estaban hechos.
Parts:
- removed U8: hm10, Connector_PinHeader_2.54mm:PinHeader_1x06_P2.54mm_Vertical, symbol hm10:hm10
- added U8: hm-10-module, symbol hm-10-bluetooth:hm-10-module
Connections:
- no-connect marks 0 -> 1
Changed lines of the file:
@@
 $EndDescr
-$Comp
-L hm10:hm10 U8
-U 1 1 61B55EEA
-P 4600 5900
-F 0 "U8" H 4878 5946 50  0000 L CNN
-F 1 "hm10" H 4878 5855 50  0000 L CNN
-F 2 "Connector_PinHeader_2.54mm:PinHeader_1x06_P2.54mm_Vertical" V 4650 5650 50  0001 L CNN
-F 3 "" H 4550 5850 50  0001 C CNN
-	1    4600 5900
-	1    0    0    -1
-$EndComp
 $Comp
 L power:+3.3V #PWR039
 U 1 1 61B55F54
-P 4150 5200
-F 0 "#PWR039" H 4150 5050 50  0001 C CNN
-F 1 "+3.3V" H 4165 5373 50  0000 C CNN
-F 2 "" H 4150 5200 50  0001 C CNN
-F 3 "" H 4150 5200 50  0001 C CNN
-	1    4150 5200
+P 3500 5450
+F 0 "#PWR039" H 3500 5300 50  0001 C CNN
+F 1 "+3.3V" H 3515 5623 50  0000 C CNN
+F 2 "" H 3500 5450 50  0001 C CNN
+F 3 "" H 3500 5450 50  0001 C CNN
+	1    3500 5450
 	1    0    0    -1
 $EndComp
@@
 L basico-rescue:GND #PWR040
 U 1 1 61B55F96
-P 4150 6250
-F 0 "#PWR040" H 4150 6000 50  0001 C CNN
-F 1 "GND" H 4155 6077 50  0000 C CNN
-F 2 "" H 4150 6250 50  0000 C CNN
-F 3 "" H 4150 6250 50  0000 C CNN
-	1    4150 6250
+P 3500 5950
+F 0 "#PWR040" H 3500 5700 50  0001 C CNN
+F 1 "GND" H 3505 5777 50  0000 C CNN
+F 2 "" H 3500 5950 50  0000 C CNN
+F 3 "" H 3500 5950 50  0000 C CNN
+	1    3500 5950
 	1    0    0    -1
 $EndComp
-Wire Wire Line
-	4150 6250 4150 6150
-Wire Wire Line
-	4150 6150 4200 6150
-Wire Wire Line
-	4200 5650 4150 5650
-Wire Wire Line
-	3800 5800 4200 5800
-Wire Wire Line
-	3800 5900 4200 5900
-Wire Wire Line
-	3800 6000 4200 6000
-Text HLabel 3800 5800 0    50   Output ~ 0
+Text HLabel 4050 5800 0    50   Output ~ 0
 BT_TX
-Text HLabel 3800 5900 0    50   Input ~ 0
+Text HLabel 4050 5900 0    50   Input ~ 0
 BT_RX
-Text HLabel 3800 6000 0    50   Output ~ 0
+Text HLabel 4050 5500 0    50   Output ~ 0
 BT_STATE
 $Comp
 L Device:C_Small C13
 U 1 1 61BB32CB
-P 4000 5450
-F 0 "C13" V 3800 5450 50  0000 C CNN
-F 1 "0.01uF" V 3900 5300 50  0000 L CNN
-F 2 "Capacitor_SMD:C_0805_2012Metric_Pad1.15x1.40mm_HandSolder" H 4000 5450 50  0001 C CNN
-F 3 "~" H 4000 5450 50  0001 C CNN
-	1    4000 5450
-	0    1    1    0
-$EndComp
-$Comp
-L basico-rescue:GND #PWR038
-U 1 1 61BB3391
-P 3800 5500
-F 0 "#PWR038" H 3800 5250 50  0001 C CNN
-F 1 "GND" H 3805 5327 50  0000 C CNN
-F 2 "" H 3800 5500 50  0000 C CNN
-F 3 "" H 3800 5500 50  0000 C CNN
-	1    3800 5500
+P 3500 5750
+F 0 "C13" H 3300 5800 50  0000 C CNN
+F 1 "0.01uF" H 3150 5700 50  0000 L CNN
+F 2 "Capacitor_SMD:C_0805_2012Metric_Pad1.15x1.40mm_HandSolder" H 3500 5750 50  0001 C CNN
+F 3 "~" H 3500 5750 50  0001 C CNN
+	1    3500 5750
 	1    0    0    -1
 $EndComp
-Wire Wire Line
-	3800 5500 3800 5450
-Wire Wire Line
-	3800 5450 3900 5450
-Wire Wire Line
-	4100 5450 4150 5450
-Wire Wire Line
-	4150 5450 4150 5650
-Connection ~ 4150 5450
-Wire Notes Line
-	3100 4900 5400 4900
-Wire Notes Line
-	5400 4900 5400 6600
-Wire Notes Line
-	5400 6600 3100 6600
 Wire Notes Line
 	3100 6600 3100 4900
@@
 Módulo Bluetooth HM-10
 Wire Wire Line
-	4150 5200 4150 5450
+	4100 5600 3500 5600
+Wire Wire Line
+	3500 5600 3500 5450
+NoConn ~ 4100 6000
+Wire Wire Line
+	3500 5600 3500 5650
+Connection ~ 3500 5600
+Wire Wire Line
+	4100 5700 3650 5700
+Wire Wire Line
+	3650 5700 3650 5900
+Wire Wire Line
+	3650 5900 3500 5900
+Wire Wire Line
+	3500 5900 3500 5850
+Wire Wire Line
+	3500 5900 3500 5950
+Connection ~ 3500 5900
+Wire Wire Line
+	4050 5500 4100 5500
+Wire Wire Line
+	4050 5800 4100 5800
+Wire Wire Line
+	4050 5900 4100 5900
+Wire Notes Line
+	5900 4900 5900 6600
+Wire Notes Line
+	3100 4900 5900 4900
+Wire Notes Line
+	3100 6600 5900 6600
+$Comp
+L hm-10-bluetooth:hm-10-module U8
+U 1 1 61D780DE
+P 4950 5750
+F 0 "U8" H 4850 6150 50  0000 L CNN
+F 1 "hm-10-module" H 4700 5350 50  0000 L CNN
+F 2 "" H 4200 5800 50  0001 C CNN
+F 3 "" H 4200 5800 50  0001 C CNN
+	1    4950 5750
+	1    0    0    -1
+$EndComp
 $EndSCHEMATC
