File: fuentes.sch (KiCad schematic (older format))
At the start: 4 parts, among them J7 BATT, U9 L7805

Commit message: Correccion de errores y se designaron huellas a casi todos los componentes
Parts:
- C15: value C_Small -> 0.01uF; footprint (none) -> Capacitor_SMD:C_0805_2012Metric_Pad1.15x1.40mm_HandSolder
- J7: footprint (none) -> TerminalBlock:TerminalBlock_bornier-2_P5.08mm
- U9: footprint (none) -> Package_TO_SOT_SMD:TO-263-3_TabPin4
Changed lines of the file:
@@
 Sheet 7 8
 Title ""
-Date ""
+Date "2021-12-19"
 Rev ""
 Comp ""
@@
 F 0 "J7" H 3520 3475 50  0000 C CNN
 F 1 "BATT" H 3520 3566 50  0000 C CNN
-F 2 "" H 3600 3800 50  0001 C CNN
+F 2 "TerminalBlock:TerminalBlock_bornier-2_P5.08mm" H 3600 3800 50  0001 C CNN
 F 3 "~" H 3600 3800 50  0001 C CNN
 	1    3600 3800
@@
 F 0 "U9" H 5150 3942 50  0000 C CNN
 F 1 "L7805" H 5150 3851 50  0000 C CNN
-F 2 "" H 5175 3550 50  0001 L CIN
+F 2 "Package_TO_SOT_SMD:TO-263-3_TabPin4" H 5175 3550 50  0001 L CIN
 F 3 "http://www.st.com/content/ccc/resource/technical/document/datasheet/41/4f/b3/b0/12/d4/47/88/CD00000444.pdf/files/CD00000444.pdf/jcr:content/translations/en.CD00000444.pdf" H 5150 3650 50  0001 C CNN
 	1    5150 3700
@@
 P 5550 4000
 F 0 "C15" H 5642 4046 50  0000 L CNN
-F 1 "C_Small" H 5642 3955 50  0000 L CNN
-F 2 "" H 5550 4000 50  0001 C CNN
+F 1 "0.01uF" H 5642 3955 50  0000 L CNN
+F 2 "Capacitor_SMD:C_0805_2012Metric_Pad1.15x1.40mm_HandSolder" H 5550 4000 50  0001 C CNN
 F 3 "~" H 5550 4000 50  0001 C CNN
 	1    5550 4000
@@
 Connection ~ 4600 3700
 Wire Wire Line
-	3900 3500 3900 3550
-Wire Wire Line
 	5550 3700 5700 3700
 $Comp
@@
 	1    0    0    -1
 $EndComp
+Wire Wire Line
+	5700 3500 5700 3700
+Wire Wire Line
+	3900 3550 3900 3700
+Wire Wire Line
+	3900 3500 3900 3550
+Connection ~ 3900 3550
+Wire Wire Line
+	4200 3550 3900 3550
+Wire Wire Line
+	4200 3500 4200 3550
 $Comp
 L power:PWR_FLAG #FLG0102
@@
 	1    0    0    -1
 $EndComp
-Wire Wire Line
-	4200 3500 4200 3550
-Wire Wire Line
-	4200 3550 3900 3550
-Connection ~ 3900 3550
-Wire Wire Line
-	3900 3550 3900 3700
-Wire Wire Line
-	5700 3500 5700 3700
 $EndSCHEMATC

Commit message: Se cambio pack de 7805 y de 9044
Parts:
- U9: footprint Package_TO_SOT_SMD:TO-263-3_TabPin4 -> Package_TO_SOT_SMD:SOT-223
Changed lines of the file:
@@
 F 0 "U9" H 5150 3942 50  0000 C CNN
 F 1 "L7805" H 5150 3851 50  0000 C CNN
-F 2 "Package_TO_SOT_SMD:TO-263-3_TabPin4" H 5175 3550 50  0001 L CIN
+F 2 "Package_TO_SOT_SMD:SOT-223" H 5175 3550 50  0001 L CIN
 F 3 "http://www.st.com/content/ccc/resource/technical/document/datasheet/41/4f/b3/b0/12/d4/47/88/CD00000444.pdf/files/CD00000444.pdf/jcr:content/translations/en.CD00000444.pdf" H 5150 3650 50  0001 C CNN
 	1    5150 3700

Commit message: Ruteado de circuito de medicion de bateria
Parts:
- added C17, C18: 0.01uF, Capacitor_SMD:C_0805_2012Metric_Pad1.15x1.40mm_HandSolder, symbol Device:C_Small
- added R12: 39k, Resistor_SMD:R_0805_2012Metric_Pad1.15x1.40mm_HandSolder, symbol Device:R_US
- added R13: 10k, Resistor_SMD:R_0805_2012Metric_Pad1.15x1.40mm_HandSolder, symbol Device:R_US
- added U10: LM358, Package_SO:SOIC-8_3.9x4.9mm_P1.27mm, symbol Amplifier_Operational:LM358
- C14: footprint (none) -> Capacitor_SMD:C_0805_2012Metric_Pad1.15x1.40mm_HandSolder
Connections:
- net labels added: V_BATT_OUT
- wire segments 20 -> 51
- no-connect marks 0 -> 1
Other:
- note added: "Conector batería y fuente 5 voltios."
- note added: "Interfaz tensión de batería y ADC"

Commit message: Comitee cambios que estaban hechos.
Parts:
- U9: footprint Package_TO_SOT_SMD:SOT-223 -> Package_TO_SOT_SMD:TO-263-3_TabPin2
Changed lines of the file:
@@
 L Connector:Screw_Terminal_01x02 J7
 U 1 1 61C4739C
-P 2950 4200
-F 0 "J7" H 2870 3875 50  0000 C CNN
-F 1 "BATT" H 2870 3966 50  0000 C CNN
-F 2 "TerminalBlock:TerminalBlock_bornier-2_P5.08mm" H 2950 4200 50  0001 C CNN
-F 3 "~" H 2950 4200 50  0001 C CNN
-	1    2950 4200
-	-1   0    0    1
+P 2950 4100
+F 0 "J7" H 2900 4300 50  0000 C CNN
+F 1 "BATT" H 2900 4200 50  0000 C CNN
+F 2 "TerminalBlock:TerminalBlock_bornier-2_P5.08mm" H 2950 4100 50  0001 C CNN
+F 3 "~" H 2950 4100 50  0001 C CNN
+	1    2950 4100
+	-1   0    0    -1
 $EndComp
 $Comp
@@
 F 0 "U9" H 4500 4342 50  0000 C CNN
 F 1 "L7805" H 4500 4251 50  0000 C CNN
-F 2 "Package_TO_SOT_SMD:SOT-223" H 4525 3950 50  0001 L CIN
+F 2 "Package_TO_SOT_SMD:TO-263-3_TabPin2" H 4525 3950 50  0001 L CIN
 F 3 "http://www.st.com/content/ccc/resource/technical/document/datasheet/41/4f/b3/b0/12/d4/47/88/CD00000444.pdf/files/CD00000444.pdf/jcr:content/translations/en.CD00000444.pdf" H 4500 4050 50  0001 C CNN
 	1    4500 4100
